Commit message: Renamed joints in the torso xacro

File: dropbear/urdf/gazebo/torso.xacro (robot description, xacro)
@@ -26,5 +26,5 @@
                 <origin xyz="-0.10115135283353449 -0.0013901114700798356 -7.263530473061719e-07" rpy="0 0 0"/>
                 <mass value="0.1475731443240637"/>
-                <inertia ixx="0.000669" iyy="0.001202" izz="0.000582" ixy="3e-05" iyz="0.0" ixz="-0.0"/>
+                <inertia ixx="0.000669" iyy="0.001202" izz="0.000582" ixy="3e-05" iyz="0.0" ixz="0.0"/>
             </inertial>
             <visual>
@@ -46,5 +46,5 @@
                 <origin xyz="-0.00311101079472062 -0.15030056139629244 3.941548639557757e-07" rpy="0 0 0"/>
                 <mass value="0.15869315430095274"/>
-                <inertia ixx="0.001188" iyy="2.2e-05" izz="0.001197" ixy="-0.000103" iyz="-0.0" ixz="-0.0"/>
+                <inertia ixx="0.001188" iyy="2.2e-05" izz="0.001197" ixy="-0.000103" iyz="0.0" ixz="0.0"/>
             </inertial>
             <visual>
@@ -66,5 +66,5 @@
                 <origin xyz="0.0021730321883888515 0.004452995163235898 0.003000367089217068" rpy="0 0 0"/>
                 <mass value="0.02600357786447301"/>
-                <inertia ixx="1.5e-05" iyy="1e-05" izz="5e-06" ixy="1e-06" iyz="-0.0" ixz="0.0"/>
+                <inertia ixx="1.5e-05" iyy="1e-05" izz="5e-06" ixy="1e-06" iyz="0.0" ixz="0.0"/>
             </inertial>
             <visual>
@@ -126,5 +126,5 @@
                 <origin xyz="-0.0032900520005997302 -0.021158555291507987 -3.4574544297422127e-06" rpy="0 0 0"/>
                 <mass value="0.030697548707811693"/>
-                <inertia ixx="2.3e-05" iyy="2.1e-05" izz="3e-06" ixy="-0.0" iyz="0.0" ixz="-0.0"/>
+                <inertia ixx="2.3e-05" iyy="2.1e-05" izz="3e-06" ixy="0.0" iyz="0.0" ixz="0.0"/>
             </inertial>
             <visual>
@@ -146,5 +146,5 @@
                 <origin xyz="0.03354545375292603 -0.02394250921487151 0.1422001419923028" rpy="0 0 0"/>
                 <mass value="0.20320755210414637"/>
-                <inertia ixx="0.000816" iyy="0.000831" izz="5.5e-05" ixy="-5e-06" iyz="0.0" ixz="-0.0"/>
+                <inertia ixx="0.000816" iyy="0.000831" izz="5.5e-05" ixy="-5e-06" iyz="0.0" ixz="0.0"/>
             </inertial>
             <visual>
@@ -206,5 +206,5 @@
                 <origin xyz="-0.0018677266631636213 -0.02751025820058717 2.3432299522951894e-07" rpy="0 0 0"/>
                 <mass value="0.024142798048081008"/>
-                <inertia ixx="1.7e-05" iyy="1.4e-05" izz="3e-06" ixy="-0.0" iyz="0.0" ixz="-0.0"/>
+                <inertia ixx="1.7e-05" iyy="1.4e-05" izz="3e-06" ixy="0.0" iyz="0.0" ixz="0.0"/>
             </inertial>
             <visual>
@@ -306,5 +306,5 @@
                 <origin xyz="-0.009999850929391957 -0.06893692335883117 0.01215561283786424" rpy="0 0 0"/>
                 <mass value="0.10579543620063496"/>
-                <inertia ixx="0.000357" iyy="1.9e-05" izz="0.000346" ixy="-0.0" iyz="6e-05" ixz="0.0"/>
+                <inertia ixx="0.000357" iyy="1.9e-05" izz="0.000346" ixy="0.0" iyz="6e-05" ixz="0.0"/>
             </inertial>
             <visual>
@@ -326,5 +326,5 @@
                 <origin xyz="-0.009999850931738746 -0.06893692336763138 -0.012155824519539338" rpy="0 0 0"/>
                 <mass value="0.10579543620063496"/>
-                <inertia ixx="0.000357" iyy="1.9e-05" izz="0.000346" ixy="-0.0" iyz="-6e-05" ixz="-0.0"/>
+                <inertia ixx="0.000357" iyy="1.9e-05" izz="0.000346" ixy="0.0" iyz="-6e-05" ixz="0.0"/>
             </inertial>
             <visual>
@@ -526,5 +526,5 @@
                 <origin xyz="0.005241809157458366 0.005244020586440523 -0.006687434993275808" rpy="0 0 0"/>
                 <mass value="0.027575447003748806"/>
-                <inertia ixx="1.2e-05" iyy="7e-06" izz="1.5e-05" ixy="-0.0" iyz="4e-06" ixz="0.0"/>
+                <inertia ixx="1.2e-05" iyy="7e-06" izz="1.5e-05" ixy="0.0" iyz="4e-06" ixz="0.0"/>
             </inertial>
             <visual>
@@ -666,5 +666,5 @@
                 <origin xyz="0.007469813078495494 0.010810047004377682 0.006925224736331809" rpy="0 0 0"/>
                 <mass value="0.02757541664931962"/>
-                <inertia ixx="1.2e-05" iyy="7e-06" izz="1.5e-05" ixy="-0.0" iyz="-4e-06" ixz="-0.0"/>
+                <inertia ixx="1.2e-05" iyy="7e-06" izz="1.5e-05" ixy="0.0" iyz="-4e-06" ixz="0.0"/>
             </inertial>
             <visual>
@@ -686,5 +686,5 @@
                 <origin xyz="-0.07015664807333664 0.00883491519637522 4.272772771568567e-07" rpy="0 0 0"/>
                 <mass value="0.10579543620063496"/>
-                <inertia ixx="3.3e-05" iyy="0.000333" izz="0.000357" ixy="8.9e-05" iyz="-0.0" ixz="0.0"/>
+                <inertia ixx="3.3e-05" iyy="0.000333" izz="0.000357" ixy="8.9e-05" iyz="0.0" ixz="0.0"/>
             </inertial>
             <visual>
@@ -726,5 +726,5 @@
                 <origin xyz="-0.07015664807242458 0.008834915186065578 3.610504858975183e-07" rpy="0 0 0"/>
                 <mass value="0.10579543620063496"/>
-                <inertia ixx="3.3e-05" iyy="0.000333" izz="0.000357" ixy="8.9e-05" iyz="-0.0" ixz="0.0"/>
+                <inertia ixx="3.3e-05" iyy="0.000333" izz="0.000357" ixy="8.9e-05" iyz="0.0" ixz="0.0"/>
             </inertial>
             <visual>
@@ -786,5 +786,5 @@
                 <origin xyz="1.7210950097740207e-07 1.474634413051179e-07 0.005697853015208351" rpy="0 0 0"/>
                 <mass value="0.13687536371193987"/>
-                <inertia ixx="2.2e-05" iyy="2.2e-05" izz="3.8e-05" ixy="-0.0" iyz="-0.0" ixz="0.0"/>
+                <inertia ixx="2.2e-05" iyy="2.2e-05" izz="3.8e-05" ixy="0.0" iyz="0.0" ixz="0.0"/>
             </inertial>
             <visual>
@@ -806,5 +806,5 @@
                 <origin xyz="1.7210949734836056e-07 1.4746372049845302e-07 -0.0024996058423814027" rpy="0 0 0"/>
                 <mass value="0.010089696045901653"/>
-                <inertia ixx="1e-06" iyy="1e-06" izz="3e-06" ixy="-0.0" iyz="-0.0" ixz="0.0"/>
+                <inertia ixx="1e-06" iyy="1e-06" izz="3e-06" ixy="0.0" iyz="0.0" ixz="0.0"/>
             </inertial>
             <visual>
@@ -846,5 +846,5 @@
                 <origin xyz="1.720538281013706e-07 1.4744714180170426e-07 -0.005697064693052395" rpy="0 0 0"/>
                 <mass value="0.13687536371193984"/>
-                <inertia ixx="2.2e-05" iyy="2.2e-05" izz="3.8e-05" ixy="-0.0" iyz="-0.0" ixz="0.0"/>
+                <inertia ixx="2.2e-05" iyy="2.2e-05" izz="3.8e-05" ixy="0.0" iyz="0.0" ixz="0.0"/>
             </inertial>
             <visual>
@@ -866,5 +866,5 @@
                 <origin xyz="1.7205387938673544e-07 1.4744684180556522e-07 0.002500394164537345" rpy="0 0 0"/>
                 <mass value="0.010089696045901642"/>
-                <inertia ixx="1e-06" iyy="1e-06" izz="3e-06" ixy="0.0" iyz="-0.0" ixz="0.0"/>
+                <inertia ixx="1e-06" iyy="1e-06" izz="3e-06" ixy="0.0" iyz="0.0" ixz="0.0"/>
             </inertial>
             <visual>
@@ -906,5 +906,5 @@
                 <origin xyz="-0.003928938015407821 -0.011151310450754293 0.008521613473048403" rpy="0 0 0"/>
                 <mass value="0.017815774190822364"/>
-                <inertia ixx="3e-06" iyy="6e-06" izz="5e-06" ixy="-0.0" iyz="1e-06" ixz="1e-06"/>
+                <inertia ixx="3e-06" iyy="6e-06" izz="5e-06" ixy="0.0" iyz="1e-06" ixz="1e-06"/>
             </inertial>
             <visual>
@@ -926,5 +926,5 @@
                 <origin xyz="-0.012355744361756071 -0.00479145026741748 0.009279912028420337" rpy="0 0 0"/>
                 <mass value="0.024414319317139412"/>
-                <inertia ixx="8e-06" iyy="1.5e-05" izz="1e-05" ixy="-0.0" iyz="1e-06" ixz="6e-06"/>
+                <inertia ixx="8e-06" iyy="1.5e-05" izz="1e-05" ixy="0.0" iyz="1e-06" ixz="6e-06"/>
             </inertial>
             <visual>
@@ -1006,5 +1006,5 @@
                 <origin xyz="-0.003928944709563065 -0.011151311045819151 -0.008520823250860177" rpy="0 0 0"/>
                 <mass value="0.01781578209705783"/>
-                <inertia ixx="3e-06" iyy="6e-06" izz="5e-06" ixy="-0.0" iyz="-1e-06" ixz="-1e-06"/>
+                <inertia ixx="3e-06" iyy="6e-06" izz="5e-06" ixy="0.0" iyz="-1e-06" ixz="-1e-06"/>
             </inertial>
             <visual>
@@ -1026,5 +1026,5 @@
                 <origin xyz="-0.012355757301481932 -0.004791417552428262 -0.009279097019659843" rpy="0 0 0"/>
                 <mass value="0.02441437178160215"/>
-                <inertia ixx="8e-06" iyy="1.5e-05" izz="1e-05" ixy="-0.0" iyz="-1e-06" ixz="-6e-06"/>
+                <inertia ixx="8e-06" iyy="1.5e-05" izz="1e-05" ixy="0.0" iyz="-1e-06" ixz="-6e-06"/>
             </inertial>
             <visual>
@@ -1106,5 +1106,5 @@
                 <origin xyz="0.022599910923873645 -0.1435763043291834 3.9415675201492917e-07" rpy="0 0 0"/>
                 <mass value="0.18514201335111086"/>
-                <inertia ixx="0.001883" iyy="2.9e-05" izz="0.001898" ixy="0.000163" iyz="-0.0" ixz="0.0"/>
+                <inertia ixx="0.001883" iyy="2.9e-05" izz="0.001898" ixy="0.000163" iyz="0.0" ixz="0.0"/>
             </inertial>
             <visual>
@@ -1186,5 +1186,5 @@
                 <origin xyz="0.020143060474379665 -0.004284392266024811 0.004022939693993005" rpy="0 0 0"/>
                 <mass value="0.04922049269032884"/>
-                <inertia ixx="1e-05" iyy="2.3e-05" izz="2.1e-05" ixy="1e-06" iyz="-0.0" ixz="-1e-06"/>
+                <inertia ixx="1e-05" iyy="2.3e-05" izz="2.1e-05" ixy="1e-06" iyz="0.0" ixz="-1e-06"/>
             </inertial>
             <visual>
@@ -1226,5 +1226,5 @@
                 <origin xyz="0.009688236645549117 -0.024337868846462135 0.0030003941618105823" rpy="0 0 0"/>
                 <mass value="0.016476308571348047"/>
-                <inertia ixx="7e-06" iyy="7e-06" izz="1e-06" ixy="0.0" iyz="0.0" ixz="-0.0"/>
+                <inertia ixx="7e-06" iyy="7e-06" izz="1e-06" ixy="0.0" iyz="0.0" ixz="0.0"/>
             </inertial>
             <visual>
@@ -1246,5 +1246,5 @@
                 <origin xyz="0.01530160397822461 0.001338830476888292 -0.032499605838198733" rpy="0 0 0"/>
                 <mass value="0.1850319786268637"/>
-                <inertia ixx="0.000158" iyy="8.5e-05" izz="0.000105" ixy="6e-06" iyz="-0.0" ixz="0.0"/>
+                <inertia ixx="0.000158" iyy="8.5e-05" izz="0.000105" ixy="6e-06" iyz="0.0" ixz="0.0"/>
             </inertial>
             <visual>
@@ -1266,5 +1266,5 @@
                 <origin xyz="0.001867733279543149 -0.027510133622699086 5.545453799354894e-07" rpy="0 0 0"/>
                 <mass value="0.024142798048081008"/>
-                <inertia ixx="1.7e-05" iyy="1.4e-05" izz="3e-06" ixy="0.0" iyz="-0.0" ixz="-0.0"/>
+                <inertia ixx="1.7e-05" iyy="1.4e-05" izz="3e-06" ixy="0.0" iyz="0.0" ixz="0.0"/>
             </inertial>
             <visual>
@@ -1366,5 +1366,5 @@
                 <origin xyz="-0.0007653000056211667 0.02219887163701692 0.020290229696044937" rpy="0 0 0"/>
                 <mass value="0.016375691601812115"/>
-                <inertia ixx="5e-06" iyy="2e-06" izz="3e-06" ixy="0.0" iyz="-0.0" ixz="-0.0"/>
+                <inertia ixx="5e-06" iyy="2e-06" izz="3e-06" ixy="0.0" iyz="0.0" ixz="0.0"/>
             </inertial>
             <visual>
@@ -1386,5 +1386,5 @@
                 <origin xyz="0.00914290933785189 0.022042515934657336 -0.020987455217608232" rpy="0 0 0"/>
                 <mass value="0.02738912858173898"/>
-                <inertia ixx="8e-06" iyy="6e-06" izz="7e-06" ixy="-0.0" iyz="0.0" ixz="-1e-06"/>
+                <inertia ixx="8e-06" iyy="6e-06" izz="7e-06" ixy="0.0" iyz="0.0" ixz="-1e-06"/>
             </inertial>
             <visual>
@@ -1406,5 +1406,5 @@
                 <origin xyz="0.014346360507995579 -0.1745967975761272 -0.01796726304975938" rpy="0 0 0"/>
                 <mass value="0.017973082329243804"/>
-                <inertia ixx="2.4e-05" iyy="9e-06" izz="1.6e-05" ixy="2e-06" iyz="-2e-06" ixz="-0.0"/>
+                <inertia ixx="2.4e-05" iyy="9e-06" izz="1.6e-05" ixy="2e-06" iyz="-2e-06" ixz="0.0"/>
             </inertial>
             <visual>
@@ -1426,5 +1426,5 @@
                 <origin xyz="0.008809576195568117 0.0007709223741320936 0.02250039415655973" rpy="0 0 0"/>
                 <mass value="0.10002696530723762"/>
-                <inertia ixx="7.8e-05" iyy="2.2e-05" izz="6.5e-05" ixy="5e-06" iyz="-0.0" ixz="0.0"/>
+                <inertia ixx="7.8e-05" iyy="2.2e-05" izz="6.5e-05" ixy="5e-06" iyz="0.0" ixz="0.0"/>
             </inertial>
             <visual>
@@ -1446,5 +1446,5 @@
                 <origin xyz="0.0011247038427605605 -0.01001039852193603 0.02444449539189178" rpy="0 0 0"/>
                 <mass value="0.017095940713325566"/>
-                <inertia ixx="8e-06" iyy="5e-06" izz="4e-06" ixy="0.0" iyz="0.0" ixz="-0.0"/>
+                <inertia ixx="8e-06" iyy="5e-06" izz="4e-06" ixy="0.0" iyz="0.0" ixz="0.0"/>
             </inertial>
             <visual>
@@ -1466,5 +1466,5 @@
                 <origin xyz="0.014278545075256333 -0.01928744128549665 0.03561120322004074" rpy="0 0 0"/>
                 <mass value="0.04300493742939915"/>
-                <inertia ixx="2.2e-05" iyy="2e-05" izz="1e-05" ixy="0.0" iyz="-0.0" ixz="-4e-06"/>
+                <inertia ixx="2.2e-05" iyy="2e-05" izz="1e-05" ixy="0.0" iyz="0.0" ixz="-4e-06"/>
             </inertial>
             <visual>
@@ -1486,5 +1486,5 @@
                 <origin xyz="-0.023929067947884963 -0.0004791829098020617 4.4941470037085374e-07" rpy="0 0 0"/>
                 <mass value="0.07961821960725156"/>
-                <inertia ixx="0.000112" iyy="7.3e-05" izz="4.4e-05" ixy="-6e-06" iyz="0.0" ixz="-0.0"/>
+                <inertia ixx="0.000112" iyy="7.3e-05" izz="4.4e-05" ixy="-6e-06" iyz="0.0" ixz="0.0"/>
             </inertial>
             <visual>
@@ -1522,377 +1522,379 @@
             </collision>
         </link> -->
-        <joint name="${prefix}_Rigid 1" type="fixed">
+        <joint name="${prefix}_Rigid1" type="fixed">
             <origin xyz="0.098178 0.07727 0.06972" rpy="0 0 0"/>
             <parent link="${prefix}_base_link"/>
             <child link="${prefix}_neck-chest-interface2_1"/>
         </joint>
-        <joint name="${prefix}_Rigid 2" type="fixed">
+        <joint name="${prefix}_Rigid2" type="fixed">
             <origin xyz="0.034406 0.025168 0.0" rpy="0 0 0"/>
             <parent link="${prefix}_neck-chest-interface2_1"/>
             <child link="${prefix}_2020_300mm_1"/>
         </joint>
-        <joint name="${prefix}_Rigid 3" type="fixed">
+        <joint name="${prefix}_Rigid3" type="fixed">
             <origin xyz="0.019924 -0.001743 -0.003" rpy="0 0 0"/>
             <parent link="${prefix}_2020_300mm_1"/>
             <child link="${prefix}_back-top__1__1"/>
         </joint>
-        <joint name="${prefix}_Rigid 4" type="fixed">
+        <joint name="${prefix}_Rigid4" type="fixed">
             <origin xyz="-0.006518 0.019009 -0.035324" rpy="0 0 0"/>
             <parent link="${prefix}_back-top__1__1"/>
             <child link="${prefix}_2020_150mm__1__1"/>
         </joint>
-        <joint name="${prefix}_Rigid 5" type="fixed">
+        <joint name="${prefix}_Rigid5" type="fixed">
             <origin xyz="-0.006518 0.019009 0.041325" rpy="0 0 0"/>
             <parent link="${prefix}_back-top__1__1"/>
             <child link="${prefix}_2020_150mm__5__1"/>
         </joint>
-        <joint name="${prefix}_Rigid 6" type="fixed">
+        <joint name="${prefix}_Rigid6" type="fixed">
             <origin xyz="0.00137 -0.030234 0.003" rpy="0 0 0"/>
             <parent link="${prefix}_back-top__1__1"/>
             <child link="${prefix}_back-middle-strap__1__1"/>
         </joint>
-        <joint name="${prefix}_Rigid 7" type="fixed">
+        <joint name="${prefix}_Rigid7" type="fixed">
             <origin xyz="-0.022632 0.055883 -0.103798" rpy="0 0 0"/>
             <parent link="${prefix}_2020_150mm__1__1"/>
             <child link="${prefix}_handle__1__1"/>
         </joint>
-        <joint name="${prefix}_Rigid 8" type="fixed">
+        <joint name="${prefix}_Rigid8" type="fixed">
             <origin xyz="-0.020657 0.051006 -0.106681" rpy="0 0 0"/>
             <parent link="${prefix}_2020_150mm__1__1"/>
             <child link="${prefix}_front-left-shoulder_1"/>
         </joint>
-        <joint name="${prefix}_Rigid 9" type="fixed">
+        <joint name="${prefix}_Rigid9" type="fixed">
             <origin xyz="-0.022632 0.055883 0.103798" rpy="0 0 0"/>
             <parent link="${prefix}_2020_150mm__5__1"/>
             <child link="${prefix}_front-right-shoulder_1"/>
         </joint>
-        <joint name="${prefix}_Rigid 10" type="fixed">
+        <joint name="${prefix}_Rigid10" type="fixed">
             <origin xyz="-0.003486 -0.039848 0.0" rpy="0 0 0"/>
             <parent link="${prefix}_back-middle-strap__1__1"/>
             <child link="${prefix}_back-bottom-strap-spine__1__1"/>
         </joint>
-        <joint name="${prefix}_Rigid 11" type="fixed">
+        <joint name="${prefix}_Rigid11" type="fixed">
             <origin xyz="-0.013813 -0.02321 -0.049813" rpy="0 0 0"/>
             <parent link="${prefix}_back-middle-strap__1__1"/>
             <child link="${prefix}_2020_100mm__4__1"/>
         </joint>
-        <joint name="${prefix}_Rigid 12" type="fixed">
+        <joint name="${prefix}_Rigid12" type="fixed">
             <origin xyz="-0.013813 -0.02321 0.049814" rpy="0 0 0"/>
             <parent link="${prefix}_back-middle-strap__1__1"/>
             <child link="${prefix}_2020_100mm__1__1"/>
         </joint>
-        <joint name="${prefix}_Rigid 13" type="fixed">
+        <joint name="${prefix}_Rigid13" type="fixed">
             <origin xyz="-0.010303 -0.042302 -0.042111" rpy="0 0 0"/>
             <parent link="${prefix}_back-bottom-strap-spine__1__1"/>
             <child link="${prefix}_2020_100mm__3__1"/>
         </joint>
-        <joint name="${prefix}_Rigid 14" type="fixed">
+        <joint name="${prefix}_Rigid14" type="fixed">
             <origin xyz="-0.010303 -0.042302 0.042112" rpy="0 0 0"/>
             <parent link="${prefix}_back-bottom-strap-spine__1__1"/>
             <child link="${prefix}_2020_100mm__2__1"/>
         </joint>
-        <joint name="${prefix}_Rigid 15" type="fixed">
+        <joint name="${prefix}_Rigid15" type="fixed">
             <origin xyz="-0.000256 -0.06214 0.002012" rpy="0 0 0"/>
             <parent link="${prefix}_front-left-shoulder_1"/>
             <child link="${prefix}_2020_200mm_1"/>
         </joint>
-        <joint name="${prefix}_Rigid 16" type="fixed">
+        <joint name="${prefix}_Rigid16" type="fixed">
             <origin xyz="0.001719 -0.067017 0.000871" rpy="0 0 0"/>
             <parent link="${prefix}_front-right-shoulder_1"/>
             <child link="${prefix}_2020_200mm__4__1"/>
         </joint>
-        <joint name="${prefix}_Rigid 17" type="fixed">
+        <joint name="${prefix}_Rigid17" type="fixed">
             <origin xyz="0.0 -0.167939 0.026566" rpy="0 0 0"/>
             <parent link="${prefix}_2020_200mm_1"/>
             <child link="${prefix}_left-front-rib-lower_1"/>
         </joint>
-        <joint name="${prefix}_Rigid 18" type="fixed">
+        <joint name="${prefix}_Rigid18" type="fixed">
             <origin xyz="0.0 -0.166897 -0.032475" rpy="0 0 0"/>
             <parent link="${prefix}_2020_200mm__4__1"/>
             <child link="${prefix}_right-front-rib-lower_1"/>
         </joint>
-        <joint name="${prefix}_Rigid 19" type="fixed">
+        <joint name="${prefix}_Rigid19" type="fixed">
             <origin xyz="-0.00055 -0.044076 0.027605" rpy="0 0 0"/>
             <parent link="${prefix}_left-front-rib-lower_1"/>
             <child link="${prefix}_2020_150mm_1"/>
         </joint>
-        <joint name="${prefix}_Rigid 20" type="fixed">
+        <joint name="${prefix}_Rigid20" type="fixed">
             <origin xyz="-0.00055 -0.045118 -0.021696" rpy="0 0 0"/>
             <parent link="${prefix}_right-front-rib-lower_1"/>
             <child link="${prefix}_2020_150mm__2__1"/>
         </joint>
-        <joint name="${prefix}_Rigid 21" type="fixed">
+        <joint name="${prefix}_Rigid21" type="fixed">
             <origin xyz="-0.006222 -0.300601 0.003" rpy="0 0 0"/>
             <parent link="${prefix}_2020_300mm_1"/>
             <child link="${prefix}_naval-strap__1__1"/>
         </joint>
-        <joint name="${prefix}_Rigid 22" type="fixed">
+        <joint name="${prefix}_Rigid22" type="fixed">
             <origin xyz="-0.013983 -0.003413 -0.06857" rpy="0 0 0"/>
             <parent link="${prefix}_2020_100mm__4__1"/>
             <child link="${prefix}_left-middle-rib_1"/>
         </joint>
-        <joint name="${prefix}_Rigid 23" type="fixed">
+        <joint name="${prefix}_Rigid23" type="fixed">
             <origin xyz="-0.053361 -0.008193 -0.014317" rpy="0 0 0"/>
             <parent link="${prefix}_left-middle-rib_1"/>
             <child link="${prefix}_2020_200mm__8__1"/>
         </joint>
-        <joint name="${prefix}_Rigid 24" type="fixed">
+        <joint name="${prefix}_Rigid24" type="fixed">
             <origin xyz="-0.168195 -0.02094 0.013451" rpy="0 0 0"/>
             <parent link="${prefix}_2020_200mm__8__1"/>
             <child link="${prefix}_rear-left-rib_1"/>
         </joint>
-        <joint name="${prefix}_Rigid 25" type="fixed">
+        <joint name="${prefix}_Rigid25" type="fixed">
             <origin xyz="0.039522 -0.033519 0.002508" rpy="0 0 0"/>
             <parent link="${prefix}_rear-left-rib_1"/>
             <child link="${prefix}_2020_200mm__2__1"/>
         </joint>
-        <joint name="${prefix}_Rigid 26" type="fixed">
+        <joint name="${prefix}_Rigid26" type="fixed">
             <origin xyz="0.158963 -0.060253 0.003046" rpy="0 0 0"/>
             <parent link="${prefix}_2020_200mm__2__1"/>
             <child link="${prefix}_left-lower-rib-side_1"/>
         </joint>
-        <joint name="${prefix}_Rigid 27" type="fixed">
+        <joint name="${prefix}_Rigid27" type="fixed">
             <origin xyz="0.029717 0.001204 -0.006361" rpy="0 0 0"/>
             <parent link="${prefix}_rear-left-rib_1"/>
             <child link="${prefix}_left-battery-mount_1"/>
         </joint>
-        <joint name="${prefix}_Rigid 28" type="fixed">
+        <joint name="${prefix}_Rigid28" type="fixed">
             <origin xyz="-0.014439 -0.00936 0.067919" rpy="0 0 0"/>
             <parent link="${prefix}_2020_100mm__1__1"/>
             <child link="${prefix}_right-middle-rib_1"/>
         </joint>
-        <joint name="${prefix}_Rigid 29" type="fixed">
+        <joint name="${prefix}_Rigid29" type="fixed">
             <origin xyz="-0.052905 -0.002246 0.014968" rpy="0 0 0"/>
             <parent link="${prefix}_right-middle-rib_1"/>
             <child link="${prefix}_2020_200mm__1__1"/>
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