Commit message: Edited -0.0 to 0.0

File: dropbear/urdf/gazebo/arm.xacro (robot description, xacro)
@@ -11,5 +11,5 @@
     <origin xyz="-6.496817022290221e-15 0.0 ${sign*0.005}" rpy="0 0 0"/>
     <mass value="0.49623462441732974"/>
-    <inertia ixx="0.000272" iyy="0.000272" izz="0.000536" ixy="-0.0" iyz="0.0" ixz="0.0"/>
+    <inertia ixx="0.000272" iyy="0.000272" izz="0.000536" ixy="0.0" iyz="0.0" ixz="0.0"/>
   </inertial>
   <visual>
@@ -31,8 +31,8 @@
     <origin xyz="-0.01659232442569455 1.1139623568467982e-07 ${sign*0.013349013943229465}" rpy="0 0 0"/>
     <mass value="0.016359268258045713"/>
-    <inertia ixx="3e-06" iyy="1e-06" izz="2e-06" ixy="-0.0" iyz="0.0" ixz="0.0"/>
-  </inertial>
-  <visual>
-    <origin xyz="-0.0 -0.0 ${sign*-0.01}" rpy="0 0 0"/>
+    <inertia ixx="3e-06" iyy="1e-06" izz="2e-06" ixy="0.0" iyz="0.0" ixz="0.0"/>
+  </inertial>
+  <visual>
+    <origin xyz="0.0 0.0 ${sign*-0.01}" rpy="0 0 0"/>
     <geometry>
       <mesh filename="package://dropbear/meshes/${folder}/shoulder-roll-al-mot_MIR1__1__1.stl" scale="0.001 0.001 0.001"/>
@@ -41,5 +41,5 @@
   </visual>
   <collision>
-    <origin xyz="-0.0 -0.0 ${sign*-0.01}" rpy="0 0 0"/>
+    <origin xyz="0.0 0.0 ${sign*-0.01}" rpy="0 0 0"/>
     <geometry>
       <mesh filename="package://dropbear/meshes/${folder}/shoulder-roll-al-mot_MIR1__1__1.stl" scale="0.001 0.001 0.001"/>
@@ -51,8 +51,8 @@
     <origin xyz="0.016592324425693906 -1.1139623519396125e-07 ${sign*0.013349013943229461}" rpy="0 0 0"/>
     <mass value="0.016359268258045713"/>
-    <inertia ixx="3e-06" iyy="1e-06" izz="2e-06" ixy="-0.0" iyz="-0.0" ixz="-0.0"/>
-  </inertial>
-  <visual>
-    <origin xyz="-0.0 -0.0 ${sign*-0.01}" rpy="0 0 0"/>
+    <inertia ixx="3e-06" iyy="1e-06" izz="2e-06" ixy="0.0" iyz="0.0" ixz="0.0"/>
+  </inertial>
+  <visual>
+    <origin xyz="0.0 0.0 ${sign*-0.01}" rpy="0 0 0"/>
     <geometry>
       <mesh filename="package://dropbear/meshes/${folder}/shoulder-roll-al-mot_MIR1__2__1.stl" scale="0.001 0.001 0.001"/>
@@ -61,5 +61,5 @@
   </visual>
   <collision>
-    <origin xyz="-0.0 -0.0 ${sign*-0.01}" rpy="0 0 0"/>
+    <origin xyz="0.0 0.0 ${sign*-0.01}" rpy="0 0 0"/>
     <geometry>
       <mesh filename="package://dropbear/meshes/${folder}/shoulder-roll-al-mot_MIR1__2__1.stl" scale="0.001 0.001 0.001"/>
@@ -74,5 +74,5 @@
   </inertial>
   <visual>
-    <origin xyz="-0.0 -0.0 ${sign*-0.11}" rpy="0 0 0"/>
+    <origin xyz="0.0 0.0 ${sign*-0.11}" rpy="0 0 0"/>
     <geometry>
       <mesh filename="package://dropbear/meshes/${folder}/yaw-cap_1.stl" scale="0.001 0.001 0.001"/>
@@ -81,5 +81,5 @@
   </visual>
   <collision>
-    <origin xyz="-0.0 -0.0 ${sign*-0.11}" rpy="0 0 0"/>
+    <origin xyz="0.0 0.0 ${sign*-0.11}" rpy="0 0 0"/>
     <geometry>
       <mesh filename="package://dropbear/meshes/${folder}/yaw-cap_1.stl" scale="0.001 0.001 0.001"/>
@@ -91,8 +91,8 @@
     <origin xyz="0.00723403458529202 -3.5971225997855074e-16 ${sign*0.0499999999999884}" rpy="0 0 0"/>
     <mass value="0.043773488134739254"/>
-    <inertia ixx="1.7e-05" iyy="8e-06" izz="1.5e-05" ixy="-0.0" iyz="-0.0" ixz="-0.0"/>
-  </inertial>
-  <visual>
-    <origin xyz="-0.0 -0.0 ${sign*-0.01}" rpy="0 0 0"/>
+    <inertia ixx="1.7e-05" iyy="8e-06" izz="1.5e-05" ixy="0.0" iyz="0.0" ixz="0.0"/>
+  </inertial>
+  <visual>
+    <origin xyz="0.0 0.0 ${sign*-0.01}" rpy="0 0 0"/>
     <geometry>
       <mesh filename="package://dropbear/meshes/${folder}/yaw-waist-adapter-motor-exal_MIR1_1.stl" scale="0.001 0.001 0.001"/>
@@ -101,5 +101,5 @@
   </visual>
   <collision>
-    <origin xyz="-0.0 -0.0 ${sign*-0.01}" rpy="0 0 0"/>
+    <origin xyz="0.0 0.0 ${sign*-0.01}" rpy="0 0 0"/>
     <geometry>
       <mesh filename="package://dropbear/meshes/${folder}/yaw-waist-adapter-motor-exal_MIR1_1.stl" scale="0.001 0.001 0.001"/>
@@ -111,5 +111,5 @@
     <origin xyz="0.007601634210069975 -0.015587999999998516 ${sign*-0.00900000000001975}" rpy="0 0 0"/>
     <mass value="0.027709236054798532"/>
-    <inertia ixx="9e-06" iyy="4e-06" izz="6e-06" ixy="0.0" iyz="-0.0" ixz="0.0"/>
+    <inertia ixx="9e-06" iyy="4e-06" izz="6e-06" ixy="0.0" iyz="0.0" ixz="0.0"/>
   </inertial>
   <visual>
@@ -131,5 +131,5 @@
     <origin xyz="-0.008272088271638172 -0.015588000000004406 ${sign*-0.008999999999990647}" rpy="0 0 0"/>
     <mass value="0.03263560284613005"/>
-    <inertia ixx="1e-05" iyy="4e-06" izz="7e-06" ixy="0.0" iyz="-0.0" ixz="0.0"/>
+    <inertia ixx="1e-05" iyy="4e-06" izz="7e-06" ixy="0.0" iyz="0.0" ixz="0.0"/>
   </inertial>
   <visual>
@@ -151,5 +151,5 @@
     <origin xyz="-0.02188091903208703 -3.219454781594442e-06 ${sign*0.0004617607023024439}" rpy="0 0 0"/>
     <mass value="0.7802158461808613"/>
-    <inertia ixx="0.001111" iyy="0.000765" izz="0.000753" ixy="0.0" iyz="-0.0" ixz="9e-06"/>
+    <inertia ixx="0.001111" iyy="0.000765" izz="0.000753" ixy="0.0" iyz="0.0" ixz="9e-06"/>
   </inertial>
   <visual>
@@ -171,5 +171,5 @@
     <origin xyz="-0.005500000000001365 -0.010394566089843876 ${sign*0.006894585665480776}" rpy="0 0 0"/>
     <mass value="0.0283879289585321"/>
-    <inertia ixx="1.2e-05" iyy="8e-06" izz="5e-06" ixy="-0.0" iyz="2e-06" ixz="0.0"/>
+    <inertia ixx="1.2e-05" iyy="8e-06" izz="5e-06" ixy="0.0" iyz="2e-06" ixz="0.0"/>
   </inertial>
   <visual>
@@ -211,5 +211,5 @@
     <origin xyz="-0.00799999999999938 -0.009999999999990211 ${sign*0.005535150009386841}" rpy="0 0 0"/>
     <mass value="0.013923035092591882"/>
-    <inertia ixx="2e-06" iyy="1e-06" izz="3e-06" ixy="-0.0" iyz="-0.0" ixz="-0.0"/>
+    <inertia ixx="2e-06" iyy="1e-06" izz="3e-06" ixy="0.0" iyz="0.0" ixz="0.0"/>
   </inertial>
   <visual>
@@ -231,5 +231,5 @@
     <origin xyz="-0.00799999999999845 -0.009999999999987075 ${sign*-0.005464849990612884}" rpy="0 0 0"/>
     <mass value="0.013923035092591882"/>
-    <inertia ixx="2e-06" iyy="1e-06" izz="3e-06" ixy="-0.0" iyz="-0.0" ixz="-0.0"/>
+    <inertia ixx="2e-06" iyy="1e-06" izz="3e-06" ixy="0.0" iyz="0.0" ixz="0.0"/>
   </inertial>
   <visual>
@@ -251,5 +251,5 @@
     <origin xyz="0.03999999999997527 0.009999999999997691 ${sign*-0.009999999999981204}" rpy="0 0 0"/>
     <mass value="0.05289771810031747"/>
-    <inertia ixx="4e-06" iyy="4.6e-05" izz="4.6e-05" ixy="-0.0" iyz="0.0" ixz="-0.0"/>
+    <inertia ixx="4e-06" iyy="4.6e-05" izz="4.6e-05" ixy="0.0" iyz="0.0" ixz="0.0"/>
   </inertial>
   <visual>
@@ -271,5 +271,5 @@
     <origin xyz="-0.04999999999998893 0.007234034585292329 ${sign*2.0539125955565396e-15}" rpy="0 0 0"/>
     <mass value="0.043773488134739254"/>
-    <inertia ixx="1.5e-05" iyy="1.7e-05" izz="8e-06" ixy="0.0" iyz="0.0" ixz="-0.0"/>
+    <inertia ixx="1.5e-05" iyy="1.7e-05" izz="8e-06" ixy="0.0" iyz="0.0" ixz="0.0"/>
   </inertial>
   <visual>
@@ -291,5 +291,5 @@
     <origin xyz="-0.01550000000000154 0.020000000000012313 ${sign*-0.007214849990613059}" rpy="0 0 0"/>
     <mass value="0.013923035092591882"/>
-    <inertia ixx="2e-06" iyy="1e-06" izz="3e-06" ixy="-0.0" iyz="-0.0" ixz="0.0"/>
+    <inertia ixx="2e-06" iyy="1e-06" izz="3e-06" ixy="0.0" iyz="0.0" ixz="0.0"/>
   </inertial>
   <visual>
@@ -311,5 +311,5 @@
     <origin xyz="-0.007736652232246094 0.010361414448293069 ${sign*0.010000000000001535}" rpy="0 0 0"/>
     <mass value="0.03345047019066647"/>
-    <inertia ixx="7e-06" iyy="6e-06" izz="6e-06" ixy="-0.0" iyz="0.0" ixz="-0.0"/>
+    <inertia ixx="7e-06" iyy="6e-06" izz="6e-06" ixy="0.0" iyz="0.0" ixz="0.0"/>
   </inertial>
   <visual>
@@ -331,5 +331,5 @@
     <origin xyz="-0.008000000000001208 -0.00999999999998867 ${sign*0.005535150009387327}" rpy="0 0 0"/>
     <mass value="0.013923035092591882"/>
-    <inertia ixx="2e-06" iyy="1e-06" izz="3e-06" ixy="-0.0" iyz="-0.0" ixz="-0.0"/>
+    <inertia ixx="2e-06" iyy="1e-06" izz="3e-06" ixy="0.0" iyz="0.0" ixz="0.0"/>
   </inertial>
   <visual>
@@ -351,5 +351,5 @@
     <origin xyz="0.004917614424534554 0.03505255276075949 ${sign*-0.025722563916740007}" rpy="0 0 0"/>
     <mass value="0.05408638346963585"/>
-    <inertia ixx="4.4e-05" iyy="1.8e-05" izz="2.6e-05" ixy="0.0" iyz="5e-06" ixz="-0.0"/>
+    <inertia ixx="4.4e-05" iyy="1.8e-05" izz="2.6e-05" ixy="0.0" iyz="5e-06" ixz="0.0"/>
   </inertial>
   <visual>
@@ -371,8 +371,8 @@
     <origin xyz="-0.007720854302206356 1.4675767796906362e-15 ${sign*-2.1421753260142395e-13}" rpy="0 0 0"/>
     <mass value="0.06058583892971603"/>
-    <inertia ixx="4.1e-05" iyy="2.2e-05" izz="2.2e-05" ixy="0.0" iyz="0.0" ixz="-0.0"/>
-  </inertial>
-  <visual>
-    <origin xyz="-0.05 -0.0 ${sign*-0.06}" rpy="0 0 0"/>
+    <inertia ixx="4.1e-05" iyy="2.2e-05" izz="2.2e-05" ixy="0.0" iyz="0.0" ixz="0.0"/>
+  </inertial>
+  <visual>
+    <origin xyz="-0.05 0.0 ${sign*-0.06}" rpy="0 0 0"/>
     <geometry>
       <mesh filename="package://dropbear/meshes/${folder}/shoulder-front-bearing-adapter_1.stl" scale="0.001 0.001 0.001"/>
@@ -381,5 +381,5 @@
   </visual>
   <collision>
-    <origin xyz="-0.05 -0.0 ${sign*-0.06}" rpy="0 0 0"/>
+    <origin xyz="-0.05 0.0 ${sign*-0.06}" rpy="0 0 0"/>
     <geometry>
       <mesh filename="package://dropbear/meshes/${folder}/shoulder-front-bearing-adapter_1.stl" scale="0.001 0.001 0.001"/>
@@ -391,8 +391,8 @@
     <origin xyz="-0.003500427124746859 9.925393840148899e-16 ${sign*6.552397513459596e-14}" rpy="0 0 0"/>
     <mass value="0.002701612602454526"/>
-    <inertia ixx="0.0" iyy="0.0" izz="0.0" ixy="0.0" iyz="-0.0" ixz="0.0"/>
-  </inertial>
-  <visual>
-    <origin xyz="-0.046172 -0.0 ${sign*-0.06}" rpy="0 0 0"/>
+    <inertia ixx="0.0" iyy="0.0" izz="0.0" ixy="0.0" iyz="0.0" ixz="0.0"/>
+  </inertial>
+  <visual>
+    <origin xyz="-0.046172 0.0 ${sign*-0.06}" rpy="0 0 0"/>
     <geometry>
       <mesh filename="package://dropbear/meshes/${folder}/skateboard-bearing__7__1.stl" scale="0.001 0.001 0.001"/>
@@ -401,5 +401,5 @@
   </visual>
   <collision>
-    <origin xyz="-0.046172 -0.0 ${sign*-0.06}" rpy="0 0 0"/>
+    <origin xyz="-0.046172 0.0 ${sign*-0.06}" rpy="0 0 0"/>
     <geometry>
       <mesh filename="package://dropbear/meshes/${folder}/skateboard-bearing__7__1.stl" scale="0.001 0.001 0.001"/>
@@ -411,5 +411,5 @@
     <origin xyz="0.009000000000008309 -0.008272088271638098 ${sign*-0.01558800000000271}" rpy="0 0 0"/>
     <mass value="0.03263560284613005"/>
-    <inertia ixx="7e-06" iyy="1e-05" izz="4e-06" ixy="0.0" iyz="0.0" ixz="-0.0"/>
+    <inertia ixx="7e-06" iyy="1e-05" izz="4e-06" ixy="0.0" iyz="0.0" ixz="0.0"/>
   </inertial>
   <visual>
@@ -451,5 +451,5 @@
     <origin xyz="-0.033978987607059224 -0.016080679496792427 ${sign*0.011692978353793536}" rpy="0 0 0"/>
     <mass value="0.037531416691209164"/>
-    <inertia ixx="6e-06" iyy="4.4e-05" izz="4.5e-05" ixy="0.0" iyz="-0.0" ixz="-0.0"/>
+    <inertia ixx="6e-06" iyy="4.4e-05" izz="4.5e-05" ixy="0.0" iyz="0.0" ixz="0.0"/>
   </inertial>
   <visual>
@@ -471,5 +471,5 @@
     <origin xyz="-0.033979393966011476 -0.017084104800040023 ${sign*0.010976523865579207}" rpy="0 0 0"/>
     <mass value="0.04634036346407298"/>
-    <inertia ixx="7e-06" iyy="2.2e-05" izz="2.4e-05" ixy="0.0" iyz="0.0" ixz="-0.0"/>
+    <inertia ixx="7e-06" iyy="2.2e-05" izz="2.4e-05" ixy="0.0" iyz="0.0" ixz="0.0"/>
   </inertial>
   <visual>
@@ -491,5 +491,5 @@
     <origin xyz="-0.00046176070351495026 -0.041996780545524526 ${sign*-0.015619080967140236}" rpy="0 0 0"/>
     <mass value="0.7802158462059968"/>
-    <inertia ixx="0.000753" iyy="0.000765" izz="0.001111" ixy="-0.0" iyz="0.0" ixz="9e-06"/>
+    <inertia ixx="0.000753" iyy="0.000765" izz="0.001111" ixy="0.0" iyz="0.0" ixz="9e-06"/>
   </inertial>
   <visual>
@@ -511,5 +511,5 @@
     <origin xyz="0.005265304298907771 -0.011277107816589804 ${sign*0.005345403003916699}" rpy="0 0 0"/>
     <mass value="0.023870437534756973"/>
-    <inertia ixx="5e-06" iyy="7e-06" izz="1.2e-05" ixy="1e-06" iyz="-0.0" ixz="0.0"/>
+    <inertia ixx="5e-06" iyy="7e-06" izz="1.2e-05" ixy="1e-06" iyz="0.0" ixz="0.0"/>
   </inertial>
   <visual>
@@ -531,5 +531,5 @@
     <origin xyz="0.005380513267402049 -0.011463196997355096 ${sign*-0.005352531151967405}" rpy="0 0 0"/>
     <mass value="0.02416670089885775"/>
-    <inertia ixx="5e-06" iyy="8e-06" izz="1.2e-05" ixy="1e-06" iyz="0.0" ixz="-0.0"/>
+    <inertia ixx="5e-06" iyy="8e-06" izz="1.2e-05" ixy="1e-06" iyz="0.0" ixz="0.0"/>
   </inertial>
   <visual>
@@ -551,5 +551,5 @@
     <origin xyz="0.0005659694928435155 -0.02118381634567837 ${sign*-0.0075641910491581615}" rpy="0 0 0"/>
     <mass value="0.010772908797143082"/>
-    <inertia ixx="3e-06" iyy="0.0" izz="3e-06" ixy="0.0" iyz="-0.0" ixz="0.0"/>
+    <inertia ixx="3e-06" iyy="0.0" izz="3e-06" ixy="0.0" iyz="0.0" ixz="0.0"/>
   </inertial>
   <visual>
@@ -571,5 +571,5 @@
     <origin xyz="-0.0015578096635837577 -0.007500647575580305 ${sign*0.016620580449611774}" rpy="0 0 0"/>
     <mass value="0.007535585538418549"/>
-    <inertia ixx="5e-06" iyy="1e-06" izz="3e-06" ixy="0.0" iyz="-0.0" ixz="-0.0"/>
+    <inertia ixx="5e-06" iyy="1e-06" izz="3e-06" ixy="0.0" iyz="0.0" ixz="0.0"/>
   </inertial>
   <visual>
@@ -591,5 +591,5 @@
     <origin xyz="0.01627296537372195 -0.009115804390395527 ${sign*-0.005357773320266886}" rpy="0 0 0"/>
     <mass value="0.027378314921932972"/>
-    <inertia ixx="6e-06" iyy="1.3e-05" izz="1.8e-05" ixy="6e-06" iyz="0.0" ixz="-0.0"/>
+    <inertia ixx="6e-06" iyy="1.3e-05" izz="1.8e-05" ixy="6e-06" iyz="0.0" ixz="0.0"/>
   </inertial>
   <visual>
@@ -611,5 +611,5 @@
     <origin xyz="3.0067933010080594e-07 -4.514541435685082e-07 ${sign*0.0025000000000662548}" rpy="0 0 0"/>
     <mass value="0.008795084983265406"/>
-    <inertia ixx="0.0" iyy="0.0" izz="0.0" ixy="-0.0" iyz="0.0" ixz="0.0"/>
+    <inertia ixx="0.0" iyy="0.0" izz="0.0" ixy="0.0" iyz="0.0" ixz="0.0"/>
   </inertial>
   <visual>
@@ -631,5 +631,5 @@
     <origin xyz="-0.004501322778096249 -0.02507818045237381 ${sign*-0.002467989334993856}" rpy="0 0 0"/>
     <mass value="0.005289691132623189"/>
-    <inertia ixx="2e-06" iyy="0.0" izz="2e-06" ixy="-0.0" iyz="0.0" ixz="0.0"/>
+    <inertia ixx="2e-06" iyy="0.0" izz="2e-06" ixy="0.0" iyz="0.0" ixz="0.0"/>
   </inertial>
   <visual>
@@ -691,5 +691,5 @@
     <origin xyz="1.5023622727816655e-07 2.8225565540385134e-07 ${sign*-0.0024999999999983508}" rpy="0 0 0"/>
     <mass value="0.008795084983265406"/>
-    <inertia ixx="0.0" iyy="0.0" izz="0.0" ixy="0.0" iyz="-0.0" ixz="0.0"/>
+    <inertia ixx="0.0" iyy="0.0" izz="0.0" ixy="0.0" iyz="0.0" ixz="0.0"/>
   </inertial>
   <visual>
@@ -771,5 +771,5 @@
     <origin xyz="-3.462138343352482e-08 6.079737324693468e-08 ${sign*0.0025000000000017786}" rpy="0 0 0"/>
     <mass value="0.008795084983265406"/>
-    <inertia ixx="0.0" iyy="0.0" izz="0.0" ixy="0.0" iyz="0.0" ixz="-0.0"/>
+    <inertia ixx="0.0" iyy="0.0" izz="0.0" ixy="0.0" iyz="0.0" ixz="0.0"/>
   </inertial>
   <visual>
@@ -811,5 +811,5 @@
     <origin xyz="-0.0005349140144733694 -0.030687105459771158 ${sign*0.004053673616640996}" rpy="0 0 0"/>
     <mass value="0.010281646529262634"/>
-    <inertia ixx="4e-06" iyy="1e-06" izz="4e-06" ixy="1e-06" iyz="-0.0" ixz="-0.0"/>
+    <inertia ixx="4e-06" iyy="1e-06" izz="4e-06" ixy="1e-06" iyz="0.0" ixz="0.0"/>
   </inertial>
   <visual>
@@ -831,5 +831,5 @@
     <origin xyz="-1.30050141874255e-07 -3.89144360235516e-07 ${sign*0.0025000000001076383}" rpy="0 0 0"/>
     <mass value="0.008795084983265406"/>
-    <inertia ixx="0.0" iyy="0.0" izz="0.0" ixy="0.0" iyz="0.0" ixz="-0.0"/>
+    <inertia ixx="0.0" iyy="0.0" izz="0.0" ixy="0.0" iyz="0.0" ixz="0.0"/>
   </inertial>
   <visual>
@@ -851,5 +851,5 @@
     <origin xyz="-1.3005014696046424e-07 -3.8914426414571324e-07 ${sign*-0.00249999999989238}" rpy="0 0 0"/>
     <mass value="0.008795084983265406"/>
-    <inertia ixx="0.0" iyy="0.0" izz="0.0" ixy="-0.0" iyz="0.0" ixz="0.0"/>
+    <inertia ixx="0.0" iyy="0.0" izz="0.0" ixy="0.0" iyz="0.0" ixz="0.0"/>
   </inertial>
   <visual>
@@ -891,5 +891,5 @@
     <origin xyz="1.239805898570201e-09 8.370368326238165e-08 ${sign*-0.002499999999896668}" rpy="0 0 0"/>
     <mass value="0.008795084983265406"/>
-    <inertia ixx="0.0" iyy="0.0" izz="0.0" ixy="0.0" iyz="-0.0" ixz="-0.0"/>
+    <inertia ixx="0.0" iyy="0.0" izz="0.0" ixy="0.0" iyz="0.0" ixz="0.0"/>
   </inertial>
   <visual>
@@ -911,5 +911,5 @@
     <origin xyz="0.0006123708628285231 -0.00038179918552844194 ${sign*-0.012000384647594495}" rpy="0 0 0"/>
     <mass value="0.0033585279582303566"/>
-    <inertia ixx="0.0" iyy="0.0" izz="0.0" ixy="-0.0" iyz="0.0" ixz="-0.0"/>
+    <inertia ixx="0.0" iyy="0.0" izz="0.0" ixy="0.0" iyz="0.0" ixz="0.0"/>
   </inertial>
   <visual>
@@ -931,5 +931,5 @@
     <origin xyz="-0.024341797177582752 -0.007557108441825444 ${sign*0.002509257258481362}" rpy="0 0 0"/>
     <mass value="0.015379539400534015"/>
-    <inertia ixx="2e-06" iyy="4e-06" izz="6e-06" ixy="0.0" iyz="-0.0" ixz="0.0"/>
+    <inertia ixx="2e-06" iyy="4e-06" izz="6e-06" ixy="0.0" iyz="0.0" ixz="0.0"/>
   </inertial>
   <visual>
@@ -951,5 +951,5 @@
     <origin xyz="-0.012981586090492152 -0.015614144505653293 ${sign*-0.04040576070339705}" rpy="0 0 0"/>
     <mass value="0.7802158462059968"/>
-    <inertia ixx="0.000765" iyy="0.001111" izz="0.000753" ixy="0.0" iyz="9e-06" ixz="-0.0"/>
+    <inertia ixx="0.000765" iyy="0.001111" izz="0.000753" ixy="0.0" iyz="9e-06" ixz="0.0"/>
   </inertial>
   <visual>
@@ -971,5 +971,5 @@
     <origin xyz="-0.0340979234925639 0.021227629310018037 ${sign*0.00035796122303764083}" rpy="0 0 0"/>
     <mass value="0.02451696606358365"/>
-    <inertia ixx="2e-06" iyy="1.3e-05" izz="1.5e-05" ixy="0.0" iyz="-0.0" ixz="0.0"/>
+    <inertia ixx="2e-06" iyy="1.3e-05" izz="1.5e-05" ixy="0.0" iyz="0.0" ixz="0.0"/>
   </inertial>
   <visual>
@@ -991,5 +991,5 @@
     <origin xyz="-0.028097214791209014 0.00645470057921349 ${sign*0.005494237705660113}" rpy="0 0 0"/>
     <mass value="0.022768388482805414"/>
-    <inertia ixx="3e-06" iyy="7e-06" izz="1e-05" ixy="1e-06" iyz="-0.0" ixz="-0.0"/>
+    <inertia ixx="3e-06" iyy="7e-06" izz="1e-05" ixy="1e-06" iyz="0.0" ixz="0.0"/>
   </inertial>
   <visual>
@@ -1011,5 +1011,5 @@
     <origin xyz="2.3269067660203202e-07 9.564553549168409e-08 ${sign*0.002500000000171587}" rpy="0 0 0"/>
     <mass value="0.008795084983265406"/>
-    <inertia ixx="0.0" iyy="0.0" izz="0.0" ixy="-0.0" iyz="0.0" ixz="0.0"/>
+    <inertia ixx="0.0" iyy="0.0" izz="0.0" ixy="0.0" iyz="0.0" ixz="0.0"/>
   </inertial>
   <visual>
@@ -1051,5 +1051,5 @@
     <origin xyz="-0.009005484461701413 -0.013346072568456768 ${sign*-0.0010043671574740468}" rpy="0 0 0"/>
     <mass value="0.016359268258045713"/>
-    <inertia ixx="1e-06" iyy="2e-06" izz="3e-06" ixy="0.0" iyz="-0.0" ixz="0.0"/>
+    <inertia ixx="1e-06" iyy="2e-06" izz="3e-06" ixy="0.0" iyz="0.0" ixz="0.0"/>
   </inertial>
   <visual>
@@ -1091,5 +1091,5 @@
     <origin xyz="-1.910406007693991e-05 -0.05000005609485908 ${sign*9.899026043314052e-14}" rpy="0 0 0"/>
     <mass value="0.052897718100317556"/>
-    <inertia ixx="4.6e-05" iyy="4e-06" izz="4.6e-05" ixy="-0.0" iyz="-0.0" ixz="-0.0"/>
+    <inertia ixx="4.6e-05" iyy="4e-06" izz="4.6e-05" ixy="0.0" iyz="0.0" ixz="0.0"/>
   </inertial>
   <visual>
@@ -1111,5 +1111,5 @@
     <origin xyz="-3.480379936662118e-05 -0.03585414266535236 ${sign*1.2044206411779279e-05}" rpy="0 0 0"/>
     <mass value="0.02056602380320786"/>
-    <inertia ixx="6e-06" iyy="1.1e-05" izz="6e-06" ixy="0.0" iyz="0.0" ixz="-0.0"/>
+    <inertia ixx="6e-06" iyy="1.1e-05" izz="6e-06" ixy="0.0" iyz="0.0" ixz="0.0"/>
   </inertial>
   <visual>
@@ -1131,5 +1131,5 @@
     <origin xyz="-0.009069915238274063 -0.023782577154890072 ${sign*-0.004850007599143107}" rpy="0 0 0"/>
     <mass value="0.05503731974130738"/>
-    <inertia ixx="9e-06" iyy="9e-06" izz="1.5e-05" ixy="-0.0" iyz="-0.0" ixz="0.0"/>
+    <inertia ixx="9e-06" iyy="9e-06" izz="1.5e-05" ixy="0.0" iyz="0.0" ixz="0.0"/>
   </inertial>
   <visual>
@@ -1151,5 +1151,5 @@
     <origin xyz="-0.004859144989096568 -0.023784135879376167 ${sign*0.009060775705327144}" rpy="0 0 0"/>
     <mass value="0.05503731974130738"/>
-    <inertia ixx="1.5e-05" iyy="9e-06" izz="9e-06" ixy="-0.0" iyz="0.0" ixz="0.0"/>
+    <inertia ixx="1.5e-05" iyy="9e-06" izz="9e-06" ixy="0.0" iyz="0.0" ixz="0.0"/>
   </inertial>
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
Commit message: edited joints names to match the ones defined in config file

File: dropbear/urdf/gazebo/arm.xacro (robot description, xacro)
@@ -1703,5 +1703,5 @@
   </joint>
 </gazebo>
-<joint name="${prefix}_Revolute55" type="revolute">
+<joint name="${prefix}_wrist_roll" type="revolute">
   <origin xyz="-0.012993 -0.036995 ${sign*-0.039944}" rpy="0 0 0"/>
   <parent link="${prefix}_RMD-X8-Pro_MIR8_MIR1__4__1"/>

File: dropbear/urdf/ros2_control/pelvicgirdle.ros2_control.xacro (robot description, xacro)
@@ -10,5 +10,5 @@
     <xacro:joint prefix="${prefix}" name="left_leg_roll" min_value="-${PI}" max_value="-${PI}">
     </xacro:joint>
-    <xacro:joint prefix="${prefix}" name="Revolute31" min_value="-${PI}" max_value="-${PI}">
+    <!-- <xacro:joint prefix="${prefix}" name="Revolute31" min_value="-${PI}" max_value="-${PI}">
     </xacro:joint>
     <xacro:joint prefix="${prefix}" name="Revolute32" min_value="-${PI}" max_value="-${PI}">
@@ -17,5 +17,5 @@
     </xacro:joint>
     <xacro:joint prefix="${prefix}" name="Revolute34" min_value="-${PI}" max_value="-${PI}">
-    </xacro:joint>
+    </xacro:joint> -->
 </xacro:macro>
 </robot>
