Commit message: edit: mesh file nameof link ${prefix}_knee-lock-2_1

File: dropbear/urdf/gazebo/leg.xacro (robot description, xacro)
@@ -497,5 +497,5 @@
                 <origin xyz="0.060896 0.378613 ${sign*-0.11}" rpy="0 0 0"/>
                 <geometry>
-                    <mesh filename="package://dropbear/meshes/${folder}/knee-lock-2_1.stl" scale="0.001 0.001 0.001"/>
+                    <mesh filename="package://dropbear/meshes/${folder}/knee-lock-2-b_1.stl" scale="0.001 0.001 0.001"/>
                 </geometry>
                 <material name="opaque191191191"/>
@@ -504,5 +504,5 @@
                 <origin xyz="0.060896 0.378613 ${sign*-0.11}" rpy="0 0 0"/>
                 <geometry>
-                    <mesh filename="package://dropbear/meshes/${folder}/knee-lock-2_1.stl" scale="0.001 0.001 0.001"/>
+                    <mesh filename="package://dropbear/meshes/${folder}/knee-lock-2-b_1.stl" scale="0.001 0.001 0.001"/>
                 </geometry>
             </collision>
