Commit message: edit: -0.0 to 0.0

File: dropbear/urdf/gazebo/leg.xacro (robot description, xacro)
@@ -35,5 +35,5 @@
             </inertial>
             <visual>
-                <origin xyz="-0.0 -0.0 ${sign*-0.01}" rpy="0 0 0"/>
+                <origin xyz="0.0 0.0 ${sign*-0.01}" rpy="0 0 0"/>
                 <geometry>
                     <mesh filename="package://dropbear/meshes/${folder}/RMD-X10-S2_MIR4__3_Stator_1.stl" scale="0.001 0.001 0.001"/>
@@ -42,5 +42,5 @@
             </visual>
             <collision>
-                <origin xyz="-0.0 -0.0 ${sign*-0.01}" rpy="0 0 0"/>
+                <origin xyz="0.0 0.0 ${sign*-0.01}" rpy="0 0 0"/>
                 <geometry>
                     <mesh filename="package://dropbear/meshes/${folder}/RMD-X10-S2_MIR4__3_Stator_1.stl" scale="0.001 0.001 0.001"/>
@@ -52,5 +52,5 @@
                 <origin xyz="0.0043331749249106155 0.00111244839801433 ${sign*0.028315467914110406}" rpy="0 0 0"/>
                 <mass value="0.024529104276010374"/>
-                <inertia ixx="1e-05" iyy="8e-06" izz="3e-06" ixy="0.0" iyz="-0.0" ixz="0.0"/>
+                <inertia ixx="1e-05" iyy="8e-06" izz="3e-06" ixy="0.0" iyz="0.0" ixz="0.0"/>
             </inertial>
             <visual>
@@ -72,5 +72,5 @@
                 <origin xyz="0.00028161841037692426 -0.004464786595415545 ${sign*0.030684539200331342}" rpy="0 0 0"/>
                 <mass value="0.024529104276010374"/>
-                <inertia ixx="8e-06" iyy="1e-05" izz="3e-06" ixy="-0.0" iyz="0.0" ixz="-0.0"/>
+                <inertia ixx="8e-06" iyy="1e-05" izz="3e-06" ixy="0.0" iyz="0.0" ixz="0.0"/>
             </inertial>
             <visual>
@@ -92,5 +92,5 @@
                 <origin xyz="-0.000281419190083107 0.004464713281593341 ${sign*0.030684532085865125}" rpy="0 0 0"/>
                 <mass value="0.024529104276010374"/>
-                <inertia ixx="8e-06" iyy="1e-05" izz="3e-06" ixy="-0.0" iyz="-0.0" ixz="0.0"/>
+                <inertia ixx="8e-06" iyy="1e-05" izz="3e-06" ixy="0.0" iyz="0.0" ixz="0.0"/>
             </inertial>
             <visual>
@@ -112,5 +112,5 @@
                 <origin xyz="-0.00433297570461362 -0.0011125217118188452 ${sign*0.02831546079961827}" rpy="0 0 0"/>
                 <mass value="0.024529104276010374"/>
-                <inertia ixx="1e-05" iyy="8e-06" izz="3e-06" ixy="0.0" iyz="0.0" ixz="-0.0"/>
+                <inertia ixx="1e-05" iyy="8e-06" izz="3e-06" ixy="0.0" iyz="0.0" ixz="0.0"/>
             </inertial>
             <visual>
@@ -132,5 +132,5 @@
                 <origin xyz="0.017145099610158858 -0.04935003665687157 ${sign*-0.004500000000001279}" rpy="0 0 0"/>
                 <mass value="0.06299639046400377"/>
-                <inertia ixx="4.2e-05" iyy="6.3e-05" izz="0.000104" ixy="3.2e-05" iyz="-0.0" ixz="0.0"/>
+                <inertia ixx="4.2e-05" iyy="6.3e-05" izz="0.000104" ixy="3.2e-05" iyz="0.0" ixz="0.0"/>
             </inertial>
             <visual>
@@ -172,8 +172,8 @@
                 <origin xyz="-0.0038111444447288256 -0.01598260549680081 ${sign*-0.008478998621304334}" rpy="0 0 0"/>
                 <mass value="0.010727755883908778"/>
-                <inertia ixx="2e-06" iyy="1e-06" izz="2e-06" ixy="-0.0" iyz="-0.0" ixz="0.0"/>
-            </inertial>
-            <visual>
-                <origin xyz="-0.053 -0.0 ${sign*-0.012}" rpy="0 0 0"/>
+                <inertia ixx="2e-06" iyy="1e-06" izz="2e-06" ixy="0.0" iyz="0.0" ixz="0.0"/>
+            </inertial>
+            <visual>
+                <origin xyz="-0.053 0.0 ${sign*-0.012}" rpy="0 0 0"/>
                 <geometry>
                     <mesh filename="package://dropbear/meshes/${folder}/knee-bend-motor-bracket-hip_1.stl" scale="0.001 0.001 0.001"/>
@@ -182,5 +182,5 @@
             </visual>
             <collision>
-                <origin xyz="-0.053 -0.0 ${sign*-0.012}" rpy="0 0 0"/>
+                <origin xyz="-0.053 0.0 ${sign*-0.012}" rpy="0 0 0"/>
                 <geometry>
                     <mesh filename="package://dropbear/meshes/${folder}/knee-bend-motor-bracket-hip_1.stl" scale="0.001 0.001 0.001"/>
@@ -192,8 +192,8 @@
                 <origin xyz="-0.0038110401177033695 -0.015982284411230948 ${sign*0.00847899862130437}" rpy="0 0 0"/>
                 <mass value="0.010727755883908778"/>
-                <inertia ixx="2e-06" iyy="1e-06" izz="2e-06" ixy="-0.0" iyz="0.0" ixz="-0.0"/>
-            </inertial>
-            <visual>
-                <origin xyz="-0.053 -0.0 ${sign*-0.071}" rpy="0 0 0"/>
+                <inertia ixx="2e-06" iyy="1e-06" izz="2e-06" ixy="0.0" iyz="0.0" ixz="0.0"/>
+            </inertial>
+            <visual>
+                <origin xyz="-0.053 0.0 ${sign*-0.071}" rpy="0 0 0"/>
                 <geometry>
                     <mesh filename="package://dropbear/meshes/${folder}/knee-bend-motor-bracket-hip__1__1.stl" scale="0.001 0.001 0.001"/>
@@ -202,5 +202,5 @@
             </visual>
             <collision>
-                <origin xyz="-0.053 -0.0 ${sign*-0.071}" rpy="0 0 0"/>
+                <origin xyz="-0.053 0.0 ${sign*-0.071}" rpy="0 0 0"/>
                 <geometry>
                     <mesh filename="package://dropbear/meshes/${folder}/knee-bend-motor-bracket-hip__1__1.stl" scale="0.001 0.001 0.001"/>
@@ -212,5 +212,5 @@
                 <origin xyz="0.01637821078173142 -0.04960639092028741 ${sign*0.02917930007753167}" rpy="0 0 0"/>
                 <mass value="1.553069048444256"/>
-                <inertia ixx="0.002856" iyy="0.002928" izz="0.003698" ixy="-0.0" iyz="-1.7e-05" ixz="0.0"/>
+                <inertia ixx="0.002856" iyy="0.002928" izz="0.003698" ixy="0.0" iyz="-1.7e-05" ixz="0.0"/>
             </inertial>
             <visual>
@@ -232,5 +232,5 @@
                 <origin xyz="-2.1161672708047696e-06 1.6410298648822375e-05 ${sign*-0.011165974681643147}" rpy="0 0 0"/>
                 <mass value="0.23611227463741877"/>
-                <inertia ixx="5.7e-05" iyy="5.7e-05" izz="7.5e-05" ixy="-0.0" iyz="-0.0" ixz="0.0"/>
+                <inertia ixx="5.7e-05" iyy="5.7e-05" izz="7.5e-05" ixy="0.0" iyz="0.0" ixz="0.0"/>
             </inertial>
             <visual>
@@ -272,5 +272,5 @@
                 <origin xyz="0.038087477180112975 0.00807344983971442 ${sign*0.00200543257018429}" rpy="0 0 0"/>
                 <mass value="0.01114960941353449"/>
-                <inertia ixx="2e-06" iyy="7e-06" izz="1e-05" ixy="-3e-06" iyz="-0.0" ixz="0.0"/>
+                <inertia ixx="2e-06" iyy="7e-06" izz="1e-05" ixy="-3e-06" iyz="0.0" ixz="0.0"/>
             </inertial>
             <visual>
@@ -292,5 +292,5 @@
                 <origin xyz="0.02831909901748353 -0.047580037015949136 ${sign*0.004499999933483212}" rpy="0 0 0"/>
                 <mass value="0.06299639046400377"/>
-                <inertia ixx="4.2e-05" iyy="6.3e-05" izz="0.000104" ixy="3.2e-05" iyz="-0.0" ixz="-0.0"/>
+                <inertia ixx="4.2e-05" iyy="6.3e-05" izz="0.000104" ixy="3.2e-05" iyz="0.0" ixz="0.0"/>
             </inertial>
             <visual>
@@ -352,5 +352,5 @@
                 <origin xyz="-9.949334274853006e-06 0.00014878773576262883 ${sign*0.013372003753055584}" rpy="0 0 0"/>
                 <mass value="0.14559026866705457"/>
-                <inertia ixx="7.3e-05" iyy="8e-05" izz="0.000138" ixy="-0.0" iyz="-2e-06" ixz="0.0"/>
+                <inertia ixx="7.3e-05" iyy="8e-05" izz="0.000138" ixy="0.0" iyz="-2e-06" ixz="0.0"/>
             </inertial>
             <visual>
@@ -372,5 +372,5 @@
                 <origin xyz="-0.00010458296907729647 0.001536971231776929 ${sign*0.010431913725907738}" rpy="0 0 0"/>
                 <mass value="0.10890019522501011"/>
-                <inertia ixx="5.3e-05" iyy="5.7e-05" izz="0.000103" ixy="-0.0" iyz="1e-06" ixz="-0.0"/>
+                <inertia ixx="5.3e-05" iyy="5.7e-05" izz="0.000103" ixy="0.0" iyz="1e-06" ixz="0.0"/>
             </inertial>
             <visual>
@@ -432,5 +432,5 @@
                 <origin xyz="-0.007433506116334768 0.1283988562731877 ${sign*0.008250058450145217}" rpy="0 0 0"/>
                 <mass value="0.03127051048143962"/>
-                <inertia ixx="4.7e-05" iyy="6e-06" izz="4.4e-05" ixy="3e-06" iyz="-0.0" ixz="0.0"/>
+                <inertia ixx="4.7e-05" iyy="6e-06" izz="4.4e-05" ixy="3e-06" iyz="0.0" ixz="0.0"/>
             </inertial>
             <visual>
@@ -452,5 +452,5 @@
                 <origin xyz="-0.0002645606062967251 0.12517110412256427 ${sign*-0.00293685000628173}" rpy="0 0 0"/>
                 <mass value="0.004721505361821494"/>
-                <inertia ixx="1e-06" iyy="0.0" izz="1e-06" ixy="0.0" iyz="0.0" ixz="-0.0"/>
+                <inertia ixx="1e-06" iyy="0.0" izz="1e-06" ixy="0.0" iyz="0.0" ixz="0.0"/>
             </inertial>
             <visual>
@@ -472,5 +472,5 @@
                 <origin xyz="0.014305292755104386 0.03576491432701612 ${sign*-0.0029994325015807732}" rpy="0 0 0"/>
                 <mass value="0.024939662437992272"/>
-                <inertia ixx="8e-06" iyy="3e-06" izz="1e-05" ixy="-1e-06" iyz="-0.0" ixz="-1e-06"/>
+                <inertia ixx="8e-06" iyy="3e-06" izz="1e-05" ixy="-1e-06" iyz="0.0" ixz="-1e-06"/>
             </inertial>
             <visual>
@@ -512,5 +512,5 @@
                 <origin xyz="-0.00043186003423186653 0.006342054694422561 ${sign*-6.298470175969406e-09}" rpy="0 0 0"/>
                 <mass value="0.03748820846896381"/>
-                <inertia ixx="2.3e-05" iyy="8e-06" izz="2.9e-05" ixy="1e-06" iyz="0.0" ixz="-0.0"/>
+                <inertia ixx="2.3e-05" iyy="8e-06" izz="2.9e-05" ixy="1e-06" iyz="0.0" ixz="0.0"/>
             </inertial>
             <visual>
@@ -532,5 +532,5 @@
                 <origin xyz="-2.900333667954502e-07 6.44297571961161e-08 ${sign*0.003500000000001016}" rpy="0 0 0"/>
                 <mass value="0.018126204213049595"/>
-                <inertia ixx="1e-06" iyy="1e-06" izz="1e-06" ixy="0.0" iyz="-0.0" ixz="0.0"/>
+                <inertia ixx="1e-06" iyy="1e-06" izz="1e-06" ixy="0.0" iyz="0.0" ixz="0.0"/>
             </inertial>
             <visual>
@@ -552,5 +552,5 @@
                 <origin xyz="-2.90033366351361e-07 6.442975647447113e-08 ${sign*-0.003499999999999018}" rpy="0 0 0"/>
                 <mass value="0.018126204213049595"/>
-                <inertia ixx="1e-06" iyy="1e-06" izz="1e-06" ixy="0.0" iyz="-0.0" ixz="0.0"/>
+                <inertia ixx="1e-06" iyy="1e-06" izz="1e-06" ixy="0.0" iyz="0.0" ixz="0.0"/>
             </inertial>
             <visual>
@@ -572,5 +572,5 @@
                 <origin xyz="0.038822812330706225 0.002017481124563625 ${sign*0.015679038691609234}" rpy="0 0 0"/>
                 <mass value="0.10127313536972944"/>
-                <inertia ixx="0.000119" iyy="0.00012" izz="0.000231" ixy="-8e-05" iyz="-2e-06" ixz="-0.0"/>
+                <inertia ixx="0.000119" iyy="0.00012" izz="0.000231" ixy="-8e-05" iyz="-2e-06" ixz="0.0"/>
             </inertial>
             <visual>
@@ -612,5 +612,5 @@
                 <origin xyz="-4.636356562559563e-09 9.929806359804116e-08 ${sign*0.004000000000000156}" rpy="0 0 0"/>
                 <mass value="0.018126204213049595"/>
-                <inertia ixx="1e-06" iyy="1e-06" izz="1e-06" ixy="-0.0" iyz="0.0" ixz="0.0"/>
+                <inertia ixx="1e-06" iyy="1e-06" izz="1e-06" ixy="0.0" iyz="0.0" ixz="0.0"/>
             </inertial>
             <visual>
@@ -632,5 +632,5 @@
                 <origin xyz="-0.0001490944286988427 -0.021355826483251888 ${sign*0.009999993701529125}" rpy="0 0 0"/>
                 <mass value="0.03748820846896381"/>
-                <inertia ixx="2.3e-05" iyy="8e-06" izz="2.9e-05" ixy="-0.0" iyz="-0.0" ixz="-0.0"/>
+                <inertia ixx="2.3e-05" iyy="8e-06" izz="2.9e-05" ixy="0.0" iyz="0.0" ixz="0.0"/>
             </inertial>
             <visual>
@@ -652,5 +652,5 @@
                 <origin xyz="-4.6363564237816846e-09 9.929819195023115e-08 ${sign*-0.003499999999999795}" rpy="0 0 0"/>
                 <mass value="0.018126204213049595"/>
-                <inertia ixx="1e-06" iyy="1e-06" izz="1e-06" ixy="0.0" iyz="0.0" ixz="-0.0"/>
+                <inertia ixx="1e-06" iyy="1e-06" izz="1e-06" ixy="0.0" iyz="0.0" ixz="0.0"/>
             </inertial>
             <visual>
@@ -712,5 +712,5 @@
                 <origin xyz="-0.00015944949609480313 -0.022838323467475854 ${sign*-0.004863339606971516}" rpy="0 0 0"/>
                 <mass value="0.03925941417972207"/>
-                <inertia ixx="2.7e-05" iyy="1e-05" izz="3.2e-05" ixy="-0.0" iyz="6e-06" ixz="0.0"/>
+                <inertia ixx="2.7e-05" iyy="1e-05" izz="3.2e-05" ixy="0.0" iyz="6e-06" ixz="0.0"/>
             </inertial>
             <visual>
@@ -732,5 +732,5 @@
                 <origin xyz="-4.636356049081414e-09 9.929806425376664e-08 ${sign*0.003500000000000149}" rpy="0 0 0"/>
                 <mass value="0.018126204213049595"/>
-                <inertia ixx="1e-06" iyy="1e-06" izz="1e-06" ixy="0.0" iyz="0.0" ixz="-0.0"/>
+                <inertia ixx="1e-06" iyy="1e-06" izz="1e-06" ixy="0.0" iyz="0.0" ixz="0.0"/>
             </inertial>
             <visual>
@@ -772,5 +772,5 @@
                 <origin xyz="-0.00032776864173092446 -0.04698371843300511 ${sign*0.017101028665118284}" rpy="0 0 0"/>
                 <mass value="0.05289771810031747"/>
-                <inertia ixx="4.6e-05" iyy="9e-06" izz="4.1e-05" ixy="-0.0" iyz="1.3e-05" ixz="0.0"/>
+                <inertia ixx="4.6e-05" iyy="9e-06" izz="4.1e-05" ixy="0.0" iyz="1.3e-05" ixz="0.0"/>
             </inertial>
             <visual>
@@ -792,5 +792,5 @@
                 <origin xyz="-0.01900539958591812 0.053069920298578654 ${sign*-0.008808113747868399}" rpy="0 0 0"/>
                 <mass value="0.044524736884465024"/>
-                <inertia ixx="1.6e-05" iyy="1.5e-05" izz="1.4e-05" ixy="0.0" iyz="-0.0" ixz="-0.0"/>
+                <inertia ixx="1.6e-05" iyy="1.5e-05" izz="1.4e-05" ixy="0.0" iyz="0.0" ixz="0.0"/>
             </inertial>
             <visual>
@@ -812,5 +812,5 @@
                 <origin xyz="-0.00011664944665303739 -0.015645331178396782 ${sign*0.008912703587378362}" rpy="0 0 0"/>
                 <mass value="0.020998682573629524"/>
-                <inertia ixx="4e-06" iyy="2e-06" izz="4e-06" ixy="-0.0" iyz="0.0" ixz="0.0"/>
+                <inertia ixx="4e-06" iyy="2e-06" izz="4e-06" ixy="0.0" iyz="0.0" ixz="0.0"/>
             </inertial>
             <visual>
@@ -832,5 +832,5 @@
                 <origin xyz="0.005201966424594279 0.03313501561044341 ${sign*-0.0014204300265370229}" rpy="0 0 0"/>
                 <mass value="0.038133616798883975"/>
-                <inertia ixx="2.4e-05" iyy="9e-06" izz="1.6e-05" ixy="-0.0" iyz="-1e-06" ixz="-0.0"/>
+                <inertia ixx="2.4e-05" iyy="9e-06" izz="1.6e-05" ixy="0.0" iyz="-1e-06" ixz="0.0"/>
             </inertial>
             <visual>
@@ -852,5 +852,5 @@
                 <origin xyz="-0.02534227251203961 0.002146310658678152 ${sign*-1.08977525614673e-09}" rpy="0 0 0"/>
                 <mass value="0.1084297628923745"/>
-                <inertia ixx="6.2e-05" iyy="6.8e-05" izz="0.000124" ixy="-1.6e-05" iyz="-0.0" ixz="0.0"/>
+                <inertia ixx="6.2e-05" iyy="6.8e-05" izz="0.000124" ixy="-1.6e-05" iyz="0.0" ixz="0.0"/>
             </inertial>
             <visual>
@@ -872,5 +872,5 @@
                 <origin xyz="1.7946537959195874e-07 1.4116536128927493e-07 ${sign*-0.0034999999999962422}" rpy="0 0 0"/>
                 <mass value="0.018126204213049595"/>
-                <inertia ixx="1e-06" iyy="1e-06" izz="1e-06" ixy="-0.0" iyz="-0.0" ixz="0.0"/>
+                <inertia ixx="1e-06" iyy="1e-06" izz="1e-06" ixy="0.0" iyz="0.0" ixz="0.0"/>
             </inertial>
             <visual>
@@ -892,5 +892,5 @@
                 <origin xyz="-3.58379128441097e-07 1.6775523914436263e-08 ${sign*-0.00349999999999652}" rpy="0 0 0"/>
                 <mass value="0.018126204213049595"/>
-                <inertia ixx="1e-06" iyy="1e-06" izz="1e-06" ixy="-0.0" iyz="0.0" ixz="0.0"/>
+                <inertia ixx="1e-06" iyy="1e-06" izz="1e-06" ixy="0.0" iyz="0.0" ixz="0.0"/>
             </inertial>
             <visual>
@@ -912,5 +912,5 @@
                 <origin xyz="1.7946537984869781e-07 1.411653617888753e-07 ${sign*0.003500000000003639}" rpy="0 0 0"/>
                 <mass value="0.018126204213049595"/>
-                <inertia ixx="1e-06" iyy="1e-06" izz="1e-06" ixy="-0.0" iyz="0.0" ixz="0.0"/>
+                <inertia ixx="1e-06" iyy="1e-06" izz="1e-06" ixy="0.0" iyz="0.0" ixz="0.0"/>
             </inertial>
             <visual>
@@ -932,5 +932,5 @@
                 <origin xyz="-3.583790006422838e-07 1.6775523192791297e-08 ${sign*0.0035000000000033615}" rpy="0 0 0"/>
                 <mass value="0.018126204213049595"/>
-                <inertia ixx="1e-06" iyy="1e-06" izz="1e-06" ixy="-0.0" iyz="0.0" ixz="-0.0"/>
+                <inertia ixx="1e-06" iyy="1e-06" izz="1e-06" ixy="0.0" iyz="0.0" ixz="0.0"/>
             </inertial>
             <visual>
@@ -952,5 +952,5 @@
                 <origin xyz="0.004788118475354965 0.11292328537245563 ${sign*-0.008977556594237712}" rpy="0 0 0"/>
                 <mass value="0.0008014552972209"/>
-                <inertia ixx="0.0" iyy="0.0" izz="0.0" ixy="0.0" iyz="0.0" ixz="-0.0"/>
+                <inertia ixx="0.0" iyy="0.0" izz="0.0" ixy="0.0" iyz="0.0" ixz="0.0"/>
             </inertial>
             <visual>
@@ -992,5 +992,5 @@
                 <origin xyz="0.023668157351731813 -0.05169650558353833 ${sign*-0.006012734795683622}" rpy="0 0 0"/>
                 <mass value="0.03733472077955106"/>
-                <inertia ixx="4.8e-05" iyy="1.2e-05" izz="5.9e-05" ixy="2.1e-05" iyz="-0.0" ixz="0.0"/>
+                <inertia ixx="4.8e-05" iyy="1.2e-05" izz="5.9e-05" ixy="2.1e-05" iyz="0.0" ixz="0.0"/>
             </inertial>
             <visual>
@@ -1012,5 +1012,5 @@
                 <origin xyz="-3.868926872693801e-07 -1.3942924020904357e-07 ${sign*-0.0034999999999952708}" rpy="0 0 0"/>
                 <mass value="0.018126204213049595"/>
-                <inertia ixx="1e-06" iyy="1e-06" izz="1e-06" ixy="-0.0" iyz="-0.0" ixz="0.0"/>
+                <inertia ixx="1e-06" iyy="1e-06" izz="1e-06" ixy="0.0" iyz="0.0" ixz="0.0"/>
             </inertial>
             <visual>
@@ -1032,5 +1032,5 @@
                 <origin xyz="-3.7732879525770313e-07 -1.6031859206844246e-07 ${sign*0.0035000000000046244}" rpy="0 0 0"/>
                 <mass value="0.018126204213049595"/>
-                <inertia ixx="1e-06" iyy="1e-06" izz="1e-06" ixy="-0.0" iyz="0.0" ixz="0.0"/>
+                <inertia ixx="1e-06" iyy="1e-06" izz="1e-06" ixy="0.0" iyz="0.0" ixz="0.0"/>
             </inertial>
             <visual>
@@ -1072,5 +1072,5 @@
                 <origin xyz="-3.2466864919797334e-07 -6.35108886037905e-08 ${sign*0.003500000000000794}" rpy="0 0 0"/>
                 <mass value="0.018126204213049595"/>
-                <inertia ixx="1e-06" iyy="1e-06" izz="1e-06" ixy="0.0" iyz="-0.0" ixz="0.0"/>
+                <inertia ixx="1e-06" iyy="1e-06" izz="1e-06" ixy="0.0" iyz="0.0" ixz="0.0"/>
             </inertial>
             <visual>
@@ -1152,5 +1152,5 @@
                 <origin xyz="-0.0017880251806005193 -0.14985476506531725 ${sign*0.018979165189555336}" rpy="0 0 0"/>
                 <mass value="0.016630111988705988"/>
-                <inertia ixx="3e-06" iyy="2e-06" izz="4e-06" ixy="-0.0" iyz="0.0" ixz="-0.0"/>
+                <inertia ixx="3e-06" iyy="2e-06" izz="4e-06" ixy="0.0" iyz="0.0" ixz="0.0"/>
             </inertial>
             <visual>
@@ -1292,5 +1292,5 @@
                 <origin xyz="0.010178865119670338 -0.006406472440295685 ${sign*-0.01082722598314824}" rpy="0 0 0"/>
                 <mass value="0.04568445868866288"/>
-                <inertia ixx="8e-06" iyy="1.6e-05" izz="2.1e-05" ixy="5e-06" iyz="-0.0" ixz="1e-06"/>
+                <inertia ixx="8e-06" iyy="1.6e-05" izz="2.1e-05" ixy="5e-06" iyz="0.0" ixz="1e-06"/>
             </inertial>
             <visual>
@@ -1372,5 +1372,5 @@
                 <origin xyz="0.0020812546237967237 -0.028665935853093183 ${sign*0.009496518706359675}" rpy="0 0 0"/>
                 <mass value="0.010036001917061667"/>
-                <inertia ixx="5e-06" iyy="1e-06" izz="5e-06" ixy="1e-06" iyz="1e-06" ixz="-0.0"/>
+                <inertia ixx="5e-06" iyy="1e-06" izz="5e-06" ixy="1e-06" iyz="1e-06" ixz="0.0"/>
             </inertial>
             <visual>
@@ -1412,5 +1412,5 @@
                 <origin xyz="0.013858476440907166 -0.012414857815914226 ${sign*0.0024342709698293996}" rpy="0 0 0"/>
                 <mass value="0.016630111988705988"/>
-                <inertia ixx="3e-06" iyy="2e-06" izz="4e-06" ixy="-0.0" iyz="0.0" ixz="-0.0"/>
+                <inertia ixx="3e-06" iyy="2e-06" izz="4e-06" ixy="0.0" iyz="0.0" ixz="0.0"/>
             </inertial>
             <visual>
@@ -1512,5 +1512,5 @@
                 <origin xyz="-7.585258199255956e-05 0.0031053120245344568 ${sign*-0.0005479105066242551}" rpy="0 0 0"/>
                 <mass value="0.08878020853187674"/>
-                <inertia ixx="7.3e-05" iyy="3.2e-05" izz="9.6e-05" ixy="1e-06" iyz="1.2e-05" ixz="-0.0"/>
+                <inertia ixx="7.3e-05" iyy="3.2e-05" izz="9.6e-05" ixy="1e-06" iyz="1.2e-05" ixz="0.0"/>
             </inertial>
             <visual>
@@ -1532,5 +1532,5 @@
                 <origin xyz="-0.017569024252099504 -0.01658185660261513 ${sign*-0.0021245329890117737}" rpy="0 0 0"/>
                 <mass value="0.025152752974316673"/>
-                <inertia ixx="4e-06" iyy="9e-06" izz="1.2e-05" ixy="-0.0" iyz="1e-06" ixz="-0.0"/>
+                <inertia ixx="4e-06" iyy="9e-06" izz="1.2e-05" ixy="0.0" iyz="1e-06" ixz="0.0"/>
             </inertial>
             <visual>
@@ -1552,5 +1552,5 @@
                 <origin xyz="-0.01767291462936746 -0.014883559282145797 ${sign*0.007519100173490473}" rpy="0 0 0"/>
                 <mass value="0.025152752974316673"/>
-                <inertia ixx="4e-06" iyy="9e-06" izz="1.2e-05" ixy="-0.0" iyz="1e-06" ixz="-0.0"/>
+                <inertia ixx="4e-06" iyy="9e-06" izz="1.2e-05" ixy="0.0" iyz="1e-06" ixz="0.0"/>
             </inertial>
             <visual>
@@ -1572,5 +1572,5 @@
                 <origin xyz="0.0012046559439662582 -0.019283720869138765 ${sign*0.013384609474228953}" rpy="0 0 0"/>
                 <mass value="0.1042453729311296"/>
-                <inertia ixx="7.2e-05" iyy="3.7e-05" izz="6.2e-05" ixy="2e-06" iyz="5e-06" ixz="-0.0"/>
+                <inertia ixx="7.2e-05" iyy="3.7e-05" izz="6.2e-05" ixy="2e-06" iyz="5e-06" ixz="0.0"/>
             </inertial>
             <visual>
@@ -1592,5 +1592,5 @@
                 <origin xyz="-0.0034942493389990142 -0.00020615226281184285 ${sign*2.1106335956616595e-05}" rpy="0 0 0"/>
                 <mass value="0.018126204213049595"/>
-                <inertia ixx="1e-06" iyy="1e-06" izz="1e-06" ixy="0.0" iyz="-0.0" ixz="-0.0"/>
+                <inertia ixx="1e-06" iyy="1e-06" izz="1e-06" ixy="0.0" iyz="0.0" ixz="0.0"/>
             </inertial>
             <visual>
@@ -1612,5 +1612,5 @@
                 <origin xyz="0.003493408858038307 0.00020522884478191283 ${sign*-2.090594191564432e-05}" rpy="0 0 0"/>
                 <mass value="0.018126204213049595"/>
-                <inertia ixx="1e-06" iyy="1e-06" izz="1e-06" ixy="0.0" iyz="-0.0" ixz="-0.0"/>
+                <inertia ixx="1e-06" iyy="1e-06" izz="1e-06" ixy="0.0" iyz="0.0" ixz="0.0"/>
             </inertial>
             <visual>
@@ -1632,5 +1632,5 @@
                 <origin xyz="0.026349579193574085 -0.0054166691408332746 ${sign*0.0010681575784079467}" rpy="0 0 0"/>
                 <mass value="0.08751895663212436"/>
-                <inertia ixx="3e-05" iyy="4.2e-05" izz="2.6e-05" ixy="0.0" iyz="-3e-06" ixz="-0.0"/>
+                <inertia ixx="3e-05" iyy="4.2e-05" izz="2.6e-05" ixy="0.0" iyz="-3e-06" ixz="0.0"/>
             </inertial>
             <visual>
@@ -1812,5 +1812,5 @@
                 <origin xyz="-0.0036931597382912906 0.004488462519170011 ${sign*-0.0008070563727921309}" rpy="0 0 0"/>
                 <mass value="0.04735315584876361"/>
-                <inertia ixx="2e-05" iyy="3.5e-05" izz="1.7e-05" ixy="-0.0" iyz="-3e-06" ixz="0.0"/>
+                <inertia ixx="2e-05" iyy="3.5e-05" izz="1.7e-05" ixy="0.0" iyz="-3e-06" ixz="0.0"/>
             </inertial>
             <visual>
@@ -1852,5 +1852,5 @@
                 <origin xyz="0.025889527959934256 0.020696987325443228 ${sign*-0.011523578858092132}" rpy="0 0 0"/>
                 <mass value="0.03465708098965354"/>
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