Commit message: edit: -0.0 to 0.0

File: dropbear/urdf/gazebo/pelvicgirdle.xacro (robot description, xacro)
@@ -7,5 +7,5 @@
                 <origin xyz="0.015013945832172346 -3.384383716609207e-07 -0.006650884466053636" rpy="0 0 0"/>
                 <mass value="0.1372183186663387"/>
-                <inertia ixx="0.000133" iyy="3.5e-05" izz="0.000117" ixy="-0.0" iyz="0.0" ixz="-1e-06"/>
+                <inertia ixx="0.000133" iyy="3.5e-05" izz="0.000117" ixy="0.0" iyz="0.0" ixz="-1e-06"/>
             </inertial>
             <visual>
@@ -27,5 +27,5 @@
                 <origin xyz="1.5368970332496623e-08 -0.015000318773633309 -4.935611415957109e-07" rpy="0 0 0"/>
                 <mass value="0.02826301085026229"/>
-                <inertia ixx="4e-06" iyy="6e-06" izz="6e-06" ixy="-0.0" iyz="0.0" ixz="0.0"/>
+                <inertia ixx="4e-06" iyy="6e-06" izz="6e-06" ixy="0.0" iyz="0.0" ixz="0.0"/>
             </inertial>
             <visual>
@@ -47,5 +47,5 @@
                 <origin xyz="1.5368829417439223e-08 0.014999681226339405 -4.935567111674644e-07" rpy="0 0 0"/>
                 <mass value="0.02826301085026229"/>
-                <inertia ixx="4e-06" iyy="6e-06" izz="6e-06" ixy="-0.0" iyz="0.0" ixz="0.0"/>
+                <inertia ixx="4e-06" iyy="6e-06" izz="6e-06" ixy="0.0" iyz="0.0" ixz="0.0"/>
             </inertial>
             <visual>
@@ -67,5 +67,5 @@
                 <origin xyz="0.0049644915520102445 0.004685619257125224 -0.023455022014617743" rpy="0 0 0"/>
                 <mass value="0.017436161627947314"/>
-                <inertia ixx="6e-06" iyy="3e-06" izz="3e-06" ixy="-0.0" iyz="1e-06" ixz="0.0"/>
+                <inertia ixx="6e-06" iyy="3e-06" izz="3e-06" ixy="0.0" iyz="1e-06" ixz="0.0"/>
             </inertial>
             <visual>
@@ -87,5 +87,5 @@
                 <origin xyz="-0.011499984065240193 -3.1877375802533657e-07 -4.935567089747739e-07" rpy="0 0 0"/>
                 <mass value="0.02345027781264517"/>
-                <inertia ixx="4e-06" iyy="3e-06" izz="3e-06" ixy="-0.0" iyz="-0.0" ixz="-0.0"/>
+                <inertia ixx="4e-06" iyy="3e-06" izz="3e-06" ixy="0.0" iyz="0.0" ixz="0.0"/>
             </inertial>
             <visual>
@@ -107,5 +107,5 @@
                 <origin xyz="-0.004457310656294178 0.003994165608435536 -0.020161167777458272" rpy="0 0 0"/>
                 <mass value="0.016984438402324765"/>
-                <inertia ixx="6e-06" iyy="4e-06" izz="2e-06" ixy="-0.0" iyz="1e-06" ixz="0.0"/>
+                <inertia ixx="6e-06" iyy="4e-06" izz="2e-06" ixy="0.0" iyz="1e-06" ixz="0.0"/>
             </inertial>
             <visual>
@@ -147,5 +147,5 @@
                 <origin xyz="-0.011499984064996444 -3.187737623311371e-07 -4.935611390699535e-07" rpy="0 0 0"/>
                 <mass value="0.02345027781264517"/>
-                <inertia ixx="4e-06" iyy="3e-06" izz="3e-06" ixy="-0.0" iyz="-0.0" ixz="-0.0"/>
+                <inertia ixx="4e-06" iyy="3e-06" izz="3e-06" ixy="0.0" iyz="0.0" ixz="0.0"/>
             </inertial>
             <visual>
@@ -207,5 +207,5 @@
                 <origin xyz="-0.009304863256996088 0.007970098995913666 -0.0163772961657776" rpy="0 0 0"/>
                 <mass value="0.01515277488114212"/>
-                <inertia ixx="6e-06" iyy="2e-06" izz="4e-06" ixy="1e-06" iyz="-0.0" ixz="-0.0"/>
+                <inertia ixx="6e-06" iyy="2e-06" izz="4e-06" ixy="1e-06" iyz="0.0" ixz="0.0"/>
             </inertial>
             <visual>
@@ -247,5 +247,5 @@
                 <origin xyz="-0.009304863257367346 -0.007970736538436926 -0.016377690952067092" rpy="0 0 0"/>
                 <mass value="0.01515277488114212"/>
-                <inertia ixx="6e-06" iyy="2e-06" izz="4e-06" ixy="-1e-06" iyz="-0.0" ixz="0.0"/>
+                <inertia ixx="6e-06" iyy="2e-06" izz="4e-06" ixy="-1e-06" iyz="0.0" ixz="0.0"/>
             </inertial>
             <visual>
@@ -267,5 +267,5 @@
                 <origin xyz="-0.00449998463110568 -0.02984731877125047 -0.04287749355892395" rpy="0 0 0"/>
                 <mass value="0.06299639046400375"/>
-                <inertia ixx="0.000104" iyy="8.6e-05" izz="1.8e-05" ixy="0.0" iyz="0.0" ixz="-0.0"/>
+                <inertia ixx="0.000104" iyy="8.6e-05" izz="1.8e-05" ixy="0.0" iyz="0.0" ixz="0.0"/>
             </inertial>
             <visual>
@@ -287,5 +287,5 @@
                 <origin xyz="0.0041146882684410385 -0.029847302967963334 -0.010695686615301458" rpy="0 0 0"/>
                 <mass value="0.026858201810092793"/>
-                <inertia ixx="1.2e-05" iyy="4e-06" izz="9e-06" ixy="-0.0" iyz="0.0" ixz="0.0"/>
+                <inertia ixx="1.2e-05" iyy="4e-06" izz="9e-06" ixy="0.0" iyz="0.0" ixz="0.0"/>
             </inertial>
             <visual>
@@ -307,5 +307,5 @@
                 <origin xyz="1.53688983067779e-08 -0.020221202063800722 0.005159838686685708" rpy="0 0 0"/>
                 <mass value="0.004432919358328168"/>
-                <inertia ixx="1e-06" iyy="0.0" izz="1e-06" ixy="0.0" iyz="-0.0" ixz="-0.0"/>
+                <inertia ixx="1e-06" iyy="0.0" izz="1e-06" ixy="0.0" iyz="0.0" ixz="0.0"/>
             </inertial>
             <visual>
@@ -327,5 +327,5 @@
                 <origin xyz="0.05000001536889755 -3.1877251323308986e-07 0.009999503884850824" rpy="0 0 0"/>
                 <mass value="0.10799999999999998"/>
-                <inertia ixx="7e-06" iyy="9.4e-05" izz="9.4e-05" ixy="-0.0" iyz="0.0" ixz="0.0"/>
+                <inertia ixx="7e-06" iyy="9.4e-05" izz="9.4e-05" ixy="0.0" iyz="0.0" ixz="0.0"/>
             </inertial>
             <visual>
@@ -347,5 +347,5 @@
                 <origin xyz="0.05000001536889753 -3.187723338210491e-07 -4.961151560678445e-07" rpy="0 0 0"/>
                 <mass value="0.10799999999999998"/>
-                <inertia ixx="7e-06" iyy="9.4e-05" izz="9.4e-05" ixy="-0.0" iyz="-0.0" ixz="0.0"/>
+                <inertia ixx="7e-06" iyy="9.4e-05" izz="9.4e-05" ixy="0.0" iyz="0.0" ixz="0.0"/>
             </inertial>
             <visual>
@@ -367,5 +367,5 @@
                 <origin xyz="0.10000001536889812 -3.1877238995670076e-07 -4.961151531812646e-07" rpy="0 0 0"/>
                 <mass value="0.10579543620063513"/>
-                <inertia ixx="9e-06" iyy="0.000357" izz="0.000357" ixy="-0.0" iyz="-0.0" ixz="0.0"/>
+                <inertia ixx="9e-06" iyy="0.000357" izz="0.000357" ixy="0.0" iyz="0.0" ixz="0.0"/>
             </inertial>
             <visual>
@@ -387,5 +387,5 @@
                 <origin xyz="-0.02314919093938346 -3.2684559186924034e-07 0.012443489936561969" rpy="0 0 0"/>
                 <mass value="0.022457820921286852"/>
-                <inertia ixx="3e-06" iyy="7e-06" izz="6e-06" ixy="-0.0" iyz="0.0" ixz="-1e-06"/>
+                <inertia ixx="3e-06" iyy="7e-06" izz="6e-06" ixy="0.0" iyz="0.0" ixz="-1e-06"/>
             </inertial>
             <visual>
@@ -427,5 +427,5 @@
                 <origin xyz="0.003364509072237204 -3.230285238048358e-07 -4.905024844070738e-07" rpy="0 0 0"/>
                 <mass value="0.02560441860614701"/>
-                <inertia ixx="5e-06" iyy="7e-06" izz="1.1e-05" ixy="-0.0" iyz="-0.0" ixz="0.0"/>
+                <inertia ixx="5e-06" iyy="7e-06" izz="1.1e-05" ixy="0.0" iyz="0.0" ixz="0.0"/>
             </inertial>
             <visual>
@@ -487,5 +487,5 @@
                 <origin xyz="1.536890698039528e-08 -3.1877150587222847e-07 -0.012305279833905003" rpy="0 0 0"/>
                 <mass value="0.019770069153948543"/>
-                <inertia ixx="4e-06" iyy="2e-06" izz="4e-06" ixy="0.0" iyz="-0.0" ixz="0.0"/>
+                <inertia ixx="4e-06" iyy="2e-06" izz="4e-06" ixy="0.0" iyz="0.0" ixz="0.0"/>
             </inertial>
             <visual>
@@ -507,5 +507,5 @@
                 <origin xyz="0.005050743795966456 0.009999681228951882 -0.010145434478224469" rpy="0 0 0"/>
                 <mass value="0.01688285985285996"/>
-                <inertia ixx="4e-06" iyy="2e-06" izz="2e-06" ixy="0.0" iyz="0.0" ixz="-0.0"/>
+                <inertia ixx="4e-06" iyy="2e-06" izz="2e-06" ixy="0.0" iyz="0.0" ixz="0.0"/>
             </inertial>
             <visual>
@@ -527,5 +527,5 @@
                 <origin xyz="-0.0049492562040334975 0.009999681228898077 -0.010145434478222026" rpy="0 0 0"/>
                 <mass value="0.01688285985285996"/>
-                <inertia ixx="4e-06" iyy="2e-06" izz="2e-06" ixy="0.0" iyz="0.0" ixz="-0.0"/>
+                <inertia ixx="4e-06" iyy="2e-06" izz="2e-06" ixy="0.0" iyz="0.0" ixz="0.0"/>
             </inertial>
             <visual>
@@ -547,5 +547,5 @@
                 <origin xyz="1.536889394915253e-08 -3.1877077208419813e-07 -0.010000496115161184" rpy="0 0 0"/>
                 <mass value="0.10799999999999998"/>
-                <inertia ixx="9.4e-05" iyy="7e-06" izz="9.4e-05" ixy="0.0" iyz="-0.0" ixz="0.0"/>
+                <inertia ixx="9.4e-05" iyy="7e-06" izz="9.4e-05" ixy="0.0" iyz="0.0" ixz="0.0"/>
             </inertial>
             <visual>
@@ -567,5 +567,5 @@
                 <origin xyz="2.0981665974084684e-08 -0.0033648124741118557 -4.918605979731261e-07" rpy="0 0 0"/>
                 <mass value="0.02560441860614701"/>
-                <inertia ixx="1.1e-05" iyy="5e-06" izz="7e-06" ixy="-0.0" iyz="-0.0" ixz="0.0"/>
+                <inertia ixx="1.1e-05" iyy="5e-06" izz="7e-06" ixy="0.0" iyz="0.0" ixz="0.0"/>
             </inertial>
             <visual>
@@ -587,5 +587,5 @@
                 <origin xyz="2.098147468265754e-08 0.0033641749325677255 -5.003697244876371e-07" rpy="0 0 0"/>
                 <mass value="0.02560441860614701"/>
-                <inertia ixx="1.1e-05" iyy="5e-06" izz="7e-06" ixy="0.0" iyz="-0.0" ixz="-0.0"/>
+                <inertia ixx="1.1e-05" iyy="5e-06" izz="7e-06" ixy="0.0" iyz="0.0" ixz="0.0"/>
             </inertial>
             <visual>
@@ -687,5 +687,5 @@
                 <origin xyz="-0.010665959312641249 -7.61455197234584e-06 1.44677919496905e-05" rpy="0 0 0"/>
                 <mass value="0.030077996769097937"/>
-                <inertia ixx="1e-05" iyy="7e-06" izz="7e-06" ixy="0.0" iyz="-0.0" ixz="-0.0"/>
+                <inertia ixx="1e-05" iyy="7e-06" izz="7e-06" ixy="0.0" iyz="0.0" ixz="0.0"/>
             </inertial>
             <visual>
@@ -707,5 +707,5 @@
                 <origin xyz="0.01276598078371094 -3.187711010987915e-07 -4.93560913139568e-07" rpy="0 0 0"/>
                 <mass value="0.043773488134739254"/>
-                <inertia ixx="1.7e-05" iyy="1.5e-05" izz="8e-06" ixy="0.0" iyz="1e-06" ixz="-0.0"/>
+                <inertia ixx="1.7e-05" iyy="1.5e-05" izz="8e-06" ixy="0.0" iyz="1e-06" ixz="0.0"/>
             </inertial>
             <visual>
@@ -727,5 +727,5 @@
                 <origin xyz="0.005000015369003186 -0.006156318771087452 -0.016914493560918786" rpy="0 0 0"/>
                 <mass value="0.020535950683961156"/>
-                <inertia ixx="7e-06" iyy="4e-06" izz="3e-06" ixy="0.0" iyz="0.0" ixz="-0.0"/>
+                <inertia ixx="7e-06" iyy="4e-06" izz="3e-06" ixy="0.0" iyz="0.0" ixz="0.0"/>
             </inertial>
             <visual>
@@ -807,5 +807,5 @@
                 <origin xyz="-0.009274838755200354 -0.027268022448470847 -0.001737513817310854" rpy="0 0 0"/>
                 <mass value="0.028033287273160054"/>
-                <inertia ixx="9e-06" iyy="6e-06" izz="7e-06" ixy="0.0" iyz="-0.0" ixz="-1e-06"/>
+                <inertia ixx="9e-06" iyy="6e-06" izz="7e-06" ixy="0.0" iyz="0.0" ixz="-1e-06"/>
             </inertial>
             <visual>
@@ -827,5 +827,5 @@
                 <origin xyz="0.004157136753358076 0.005209080370864566 -0.02954422733259171" rpy="0 0 0"/>
                 <mass value="0.022555609719694947"/>
-                <inertia ixx="1e-05" iyy="6e-06" izz="4e-06" ixy="0.0" iyz="0.0" ixz="-0.0"/>
+                <inertia ixx="1e-05" iyy="6e-06" izz="4e-06" ixy="0.0" iyz="0.0" ixz="0.0"/>
             </inertial>
             <visual>
@@ -847,5 +847,5 @@
                 <origin xyz="0.0041571367533579096 0.005209080370864372 -0.029544227332592266" rpy="0 0 0"/>
                 <mass value="0.022555609719694947"/>
-                <inertia ixx="1e-05" iyy="6e-06" izz="4e-06" ixy="0.0" iyz="0.0" ixz="-0.0"/>
+                <inertia ixx="1e-05" iyy="6e-06" izz="4e-06" ixy="0.0" iyz="0.0" ixz="0.0"/>
             </inertial>
             <visual>
@@ -867,5 +867,5 @@
                 <origin xyz="0.01000001604236285 -0.0016471342297867397 0.009338192977970172" rpy="0 0 0"/>
                 <mass value="0.011013373716250049"/>
-                <inertia ixx="2e-06" iyy="1e-06" izz="2e-06" ixy="0.0" iyz="-0.0" ixz="0.0"/>
+                <inertia ixx="2e-06" iyy="1e-06" izz="2e-06" ixy="0.0" iyz="0.0" ixz="0.0"/>
             </inertial>
             <visual>
@@ -927,5 +927,5 @@
                 <origin xyz="0.05300006756213727 0.002535021218337402 -0.017170296793771855" rpy="0 0 0"/>
                 <mass value="1.174088575802461"/>
-                <inertia ixx="0.001602" iyy="0.00167" izz="0.002602" ixy="-0.0" iyz="-0.000178" ixz="-0.0"/>
+                <inertia ixx="0.001602" iyy="0.00167" izz="0.002602" ixy="0.0" iyz="-0.000178" ixz="0.0"/>
             </inertial>
             <visual>
@@ -947,5 +947,5 @@
                 <origin xyz="-0.005073926852487115 -0.0004083027309976228 -0.006087188505683183" rpy="0 0 0"/>
                 <mass value="0.013793283494451192"/>
-                <inertia ixx="3e-06" iyy="3e-06" izz="5e-06" ixy="-2e-06" iyz="-0.0" ixz="-0.0"/>
+                <inertia ixx="3e-06" iyy="3e-06" izz="5e-06" ixy="-2e-06" iyz="0.0" ixz="0.0"/>
             </inertial>
             <visual>
@@ -967,5 +967,5 @@
                 <origin xyz="0.005228251371043061 0.011836701255534987 0.007672233029588471" rpy="0 0 0"/>
                 <mass value="0.017182715926445345"/>
-                <inertia ixx="3e-06" iyy="2e-06" izz="5e-06" ixy="1e-06" iyz="-0.0" ixz="0.0"/>
+                <inertia ixx="3e-06" iyy="2e-06" izz="5e-06" ixy="1e-06" iyz="0.0" ixz="0.0"/>
             </inertial>
             <visual>
@@ -987,5 +987,5 @@
                 <origin xyz="0.005228251371024797 0.013747165395658636 -0.003160730160940317" rpy="0 0 0"/>
                 <mass value="0.017182715926445345"/>
-                <inertia ixx="3e-06" iyy="2e-06" izz="5e-06" ixy="1e-06" iyz="-0.0" ixz="0.0"/>
+                <inertia ixx="3e-06" iyy="2e-06" izz="5e-06" ixy="1e-06" iyz="0.0" ixz="0.0"/>
             </inertial>
             <visual>
@@ -1027,5 +1027,5 @@
                 <origin xyz="-8.723622045594265e-06 -0.0018885018109361107 0.010799035281507052" rpy="0 0 0"/>
                 <mass value="0.027281477204810733"/>
-                <inertia ixx="6e-06" iyy="6e-06" izz="8e-06" ixy="-0.0" iyz="-0.0" ixz="-0.0"/>
+                <inertia ixx="6e-06" iyy="6e-06" izz="8e-06" ixy="0.0" iyz="0.0" ixz="0.0"/>
             </inertial>
             <visual>
@@ -1047,5 +1047,5 @@
                 <origin xyz="1.5368970672502424e-08 0.00868260797978701 -0.04924027374717088" rpy="0 0 0"/>
                 <mass value="0.05289771810031747"/>
-                <inertia ixx="4.6e-05" iyy="4.5e-05" izz="6e-06" ixy="0.0" iyz="7e-06" ixz="-0.0"/>
+                <inertia ixx="4.6e-05" iyy="4.5e-05" izz="6e-06" ixy="0.0" iyz="7e-06" ixz="0.0"/>
             </inertial>
             <visual>
@@ -1067,5 +1067,5 @@
                 <origin xyz="0.01657265300759825 0.004034163613513886 -0.022877676923640844" rpy="0 0 0"/>
                 <mass value="0.02887084772533379"/>
-                <inertia ixx="9e-06" iyy="6e-06" izz="4e-06" ixy="-0.0" iyz="0.0" ixz="0.0"/>
+                <inertia ixx="9e-06" iyy="6e-06" izz="4e-06" ixy="0.0" iyz="0.0" ixz="0.0"/>
             </inertial>
             <visual>
@@ -1087,5 +1087,5 @@
                 <origin xyz="-0.016572622269602787 0.004034177703166858 -0.022877674439242768" rpy="0 0 0"/>
                 <mass value="0.02887084772533379"/>
-                <inertia ixx="9e-06" iyy="6e-06" izz="4e-06" ixy="0.0" iyz="0.0" ixz="-0.0"/>
+                <inertia ixx="9e-06" iyy="6e-06" izz="4e-06" ixy="0.0" iyz="0.0" ixz="0.0"/>
             </inertial>
             <visual>
@@ -1107,5 +1107,5 @@
                 <origin xyz="1.4713597788068578e-08 0.026187946354894187 -0.010407331087171512" rpy="0 0 0"/>
                 <mass value="0.008295431917978503"/>
-                <inertia ixx="1e-06" iyy="1e-06" izz="1e-06" ixy="0.0" iyz="-0.0" ixz="0.0"/>
+                <inertia ixx="1e-06" iyy="1e-06" izz="1e-06" ixy="0.0" iyz="0.0" ixz="0.0"/>
             </inertial>
             <visual>
@@ -1127,5 +1127,5 @@
                 <origin xyz="1.5368992366954215e-08 -0.01233356181134436 0.028288394269538386" rpy="0 0 0"/>
                 <mass value="0.043773488134739254"/>
-                <inertia ixx="8e-06" iyy="1.7e-05" izz="1.5e-05" ixy="-0.0" iyz="0.0" ixz="0.0"/>
+                <inertia ixx="8e-06" iyy="1.7e-05" izz="1.5e-05" ixy="0.0" iyz="0.0" ixz="0.0"/>
             </inertial>
             <visual>
@@ -1147,5 +1147,5 @@
                 <origin xyz="-0.015587984631046943 0.00648668782886265 -0.007994706141802255" rpy="0 0 0"/>
                 <mass value="0.020535950683961156"/>
-                <inertia ixx="3e-06" iyy="6e-06" izz="4e-06" ixy="-0.0" iyz="0.0" ixz="-0.0"/>
+                <inertia ixx="3e-06" iyy="6e-06" izz="4e-06" ixy="0.0" iyz="0.0" ixz="0.0"/>
             </inertial>
             <visual>
@@ -1167,5 +1167,5 @@
                 <origin xyz="-0.01558798463097628 -0.003361622291394334 -0.009731633249791649" rpy="0 0 0"/>
                 <mass value="0.020535950683961156"/>
-                <inertia ixx="3e-06" iyy="6e-06" izz="4e-06" ixy="-0.0" iyz="0.0" ixz="-0.0"/>
+                <inertia ixx="3e-06" iyy="6e-06" izz="4e-06" ixy="0.0" iyz="0.0" ixz="0.0"/>
             </inertial>
             <visual>
@@ -1187,5 +1187,5 @@
                 <origin xyz="-0.015587859166047092 -0.0008996427037845367 -0.009297208589254646" rpy="0 0 0"/>
                 <mass value="0.01026797534198055"/>
-                <inertia ixx="1e-06" iyy="3e-06" izz="2e-06" ixy="0.0" iyz="0.0" ixz="-0.0"/>
+                <inertia ixx="1e-06" iyy="3e-06" izz="2e-06" ixy="0.0" iyz="0.0" ixz="0.0"/>
             </inertial>
             <visual>
@@ -1247,5 +1247,5 @@
                 <origin xyz="-0.010665959312859588 2.572880747566189e-06 1.589878415281243e-05" rpy="0 0 0"/>
                 <mass value="0.030077996769097937"/>
-                <inertia ixx="1e-05" iyy="7e-06" izz="7e-06" ixy="-0.0" iyz="0.0" ixz="-0.0"/>
+                <inertia ixx="1e-05" iyy="7e-06" izz="7e-06" ixy="0.0" iyz="0.0" ixz="0.0"/>
             </inertial>
             <visual>
@@ -1287,5 +1287,5 @@
                 <origin xyz="0.005000015368784895 -0.011570318771084437 -0.013788493556942394" rpy="0 0 0"/>
                 <mass value="0.020535950683961156"/>
-                <inertia ixx="7e-06" iyy="4e-06" izz="3e-06" ixy="0.0" iyz="-0.0" ixz="0.0"/>
+                <inertia ixx="7e-06" iyy="4e-06" izz="3e-06" ixy="0.0" iyz="0.0" ixz="0.0"/>
             </inertial>
             <visual>
@@ -1307,5 +1307,5 @@
                 <origin xyz="-0.009999984631215104 0.018711681228903265 -0.0032994935569432005" rpy="0 0 0"/>
                 <mass value="0.10799999999999998"/>
-                <inertia ixx="9.4e-05" iyy="1e-05" izz="9.1e-05" ixy="0.0" iyz="1.5e-05" ixz="-0.0"/>
+                <inertia ixx="9.4e-05" iyy="1e-05" izz="9.1e-05" ixy="0.0" iyz="1.5e-05" ixz="0.0"/>
             </inertial>
             <visual>
@@ -1327,5 +1327,5 @@
                 <origin xyz="1.5368768244150566e-08 -0.049240318771098336 0.00868250644305707" rpy="0 0 0"/>
                 <mass value="0.05289771810031747"/>
-                <inertia ixx="4.6e-05" iyy="6e-06" izz="4.5e-05" ixy="0.0" iyz="7e-06" ixz="-0.0"/>
+                <inertia ixx="4.6e-05" iyy="6e-06" izz="4.5e-05" ixy="0.0" iyz="7e-06" ixz="0.0"/>
             </inertial>
             <visual>
@@ -1347,5 +1347,5 @@
                 <origin xyz="1.536867939855302e-08 6.8879795873944e-08 9.756131469362828e-08" rpy="0 0 0"/>
                 <mass value="0.05289771810031747"/>
-                <inertia ixx="4.6e-05" iyy="6e-06" izz="4.5e-05" ixy="0.0" iyz="7e-06" ixz="-0.0"/>
+                <inertia ixx="4.6e-05" iyy="6e-06" izz="4.5e-05" ixy="0.0" iyz="7e-06" ixz="0.0"/>
             </inertial>
             <visual>
@@ -1367,5 +1367,5 @@
                 <origin xyz="1.730971942170978e-08 0.027257052209767166 -0.003781036214674016" rpy="0 0 0"/>
                 <mass value="0.043764820713222324"/>
-                <inertia ixx="1.4e-05" iyy="1.5e-05" izz="1.6e-05" ixy="-0.0" iyz="0.0" ixz="-0.0"/>
+                <inertia ixx="1.4e-05" iyy="1.5e-05" izz="1.6e-05" ixy="0.0" iyz="0.0" ixz="0.0"/>
             </inertial>
             <visual>
@@ -1387,5 +1387,5 @@
                 <origin xyz="0.004157136752864998 -0.005209717912239634 -0.029544227323636985" rpy="0 0 0"/>
                 <mass value="0.022555609719694947"/>
-                <inertia ixx="1e-05" iyy="6e-06" izz="4e-06" ixy="0.0" iyz="-0.0" ixz="0.0"/>
+                <inertia ixx="1e-05" iyy="6e-06" izz="4e-06" ixy="0.0" iyz="0.0" ixz="0.0"/>
             </inertial>
             <visual>
@@ -1407,5 +1407,5 @@
                 <origin xyz="-0.0041571060155706635 -0.005209717912184789 -0.029544227323650085" rpy="0 0 0"/>
                 <mass value="0.022555609719694947"/>
-                <inertia ixx="1e-05" iyy="6e-06" izz="4e-06" ixy="0.0" iyz="-0.0" ixz="0.0"/>
+                <inertia ixx="1e-05" iyy="6e-06" izz="4e-06" ixy="0.0" iyz="0.0" ixz="0.0"/>
             </inertial>
             <visual>
@@ -1447,5 +1447,5 @@
                 <origin xyz="0.010000016041882609 0.001646489975612779 0.009338194170572856" rpy="0 0 0"/>
                 <mass value="0.011013373716250049"/>
-                <inertia ixx="2e-06" iyy="1e-06" izz="2e-06" ixy="0.0" iyz="0.0" ixz="-0.0"/>
+                <inertia ixx="2e-06" iyy="1e-06" izz="2e-06" ixy="0.0" iyz="0.0" ixz="0.0"/>
             </inertial>
             <visual>
@@ -1507,5 +1507,5 @@
                 <origin xyz="0.0428779631756421 0.02814434123985871 -0.022580296789184773" rpy="0 0 0"/>
                 <mass value="1.1740885758024595"/>
-                <inertia ixx="0.001602" iyy="0.00167" izz="0.002602" ixy="-0.0" iyz="0.000178" ixz="0.0"/>
+                <inertia ixx="0.001602" iyy="0.00167" izz="0.002602" ixy="0.0" iyz="0.000178" ixz="0.0"/>
             </inertial>
             <visual>
@@ -1527,5 +1527,5 @@
                 <origin xyz="-0.005073925582805672 0.0004076645392949302 -0.00608718879908049" rpy="0 0 0"/>
                 <mass value="0.013793283930020089"/>
-                <inertia ixx="3e-06" iyy="3e-06" izz="5e-06" ixy="2e-06" iyz="0.0" ixz="-0.0"/>
+                <inertia ixx="3e-06" iyy="3e-06" izz="5e-06" ixy="2e-06" iyz="0.0" ixz="0.0"/>
             </inertial>
             <visual>
@@ -1587,5 +1587,5 @@
                 <origin xyz="-0.0015478476609870478 -0.01279789904450368 -0.016020226205955224" rpy="0 0 0"/>
                 <mass value="0.02289025400758011"/>
-                <inertia ixx="5e-06" iyy="3e-06" izz="3e-06" ixy="-0.0" iyz="-0.0" ixz="0.0"/>
+                <inertia ixx="5e-06" iyy="3e-06" izz="3e-06" ixy="0.0" iyz="0.0" ixz="0.0"/>
             </inertial>
             <visual>
@@ -1607,5 +1607,5 @@
                 <origin xyz="8.754359823594238e-06 0.0018888642697480248 0.010799035285952774" rpy="0 0 0"/>
                 <mass value="0.027281477204810733"/>
-                <inertia ixx="6e-06" iyy="6e-06" izz="8e-06" ixy="-0.0" iyz="0.0" ixz="0.0"/>
+                <inertia ixx="6e-06" iyy="6e-06" izz="8e-06" ixy="0.0" iyz="0.0" ixz="0.0"/>
             </inertial>
             <visual>
@@ -1627,5 +1627,5 @@
                 <origin xyz="1.5368764684497993e-08 -0.008682245517031392 -0.04924027374342238" rpy="0 0 0"/>
                 <mass value="0.05289771810031747"/>
-                <inertia ixx="4.6e-05" iyy="4.5e-05" izz="6e-06" ixy="-0.0" iyz="-7e-06" ixz="-0.0"/>
+                <inertia ixx="4.6e-05" iyy="4.5e-05" izz="6e-06" ixy="0.0" iyz="-7e-06" ixz="0.0"/>
             </inertial>
             <visual>
@@ -1647,5 +1647,5 @@
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