Commit message: comment out base link definition in leg.xacro

File: dropbear-humanoid-robot/dropbear/urdf/gazebo/leg.xacro (robot description, xacro)
@@ -8,5 +8,5 @@
    -->
     <xacro:macro name="leg_macro" params="prefix folder parent sign *origin">
-        <link name="${prefix}_base_link">
+        <!-- <link name="${prefix}_base_link">
             <inertial>
                 <origin xyz="-2.1374041718990718e-14 0.0 ${sign*0.005}" rpy="0 0 0"/>
@@ -27,5 +27,5 @@
                 </geometry>
             </collision>
-        </link>
+        </link> -->
         <link name="${prefix}_RMD-X10-S2_MIR4__3_Stator_1">
             <inertial>
