Commit message: add dynamics properties to joints in pelvicgirdle.xacro and update joint limits in arm.ros2_control.xacro

File: dropbear-humanoid-robot/dropbear/urdf/gazebo/pelvicgirdle.xacro (robot description, xacro)
@@ -1972,4 +1972,5 @@
             <axis xyz="1.0 0.0 0.0"/>
             <limit upper="${PI}" lower="${-PI}" velocity="10.0" effort="10.0"/>
+            <dynamics damping="10.0" friction="0.50"/>
         </joint>
         <joint name="${prefix}_Rigid36" type="fixed">
@@ -2059,4 +2060,5 @@
             <axis xyz="0.0 0.173648 -0.984808"/>
             <limit upper="${PI}" lower="${-PI}" velocity="10.0" effort="10.0"/>
+            <dynamics damping="10.0" friction="0.50"/>
         </joint>
         <joint name="${prefix}_Rigid53" type="fixed">
@@ -2116,4 +2118,5 @@
             <axis xyz="1.0 0.0 0.0"/>
             <limit upper="${PI}" lower="${-PI}" velocity="10.0" effort="10.0"/>
+            <dynamics damping="10.0" friction="0.50"/>
         </joint>
         <joint name="${prefix}_Rigid64" type="fixed">
@@ -2208,4 +2211,5 @@
             <axis xyz="0.0 -0.173648 -0.984808"/>
             <limit upper="${PI}" lower="${-PI}" velocity="10.0" effort="10.0"/>
+            <dynamics damping="10.0" friction="0.50"/>
         </joint>
         <joint name="${prefix}_Rigid82" type="fixed">
