Commit message: update arm.xacro to use dynamic axis values for joint configurations

File: dropbear-humanoid-robot/dropbear/urdf/gazebo/arm.xacro (robot description, xacro)
@@ -1407,5 +1407,5 @@
       <parent link="${prefix}_shoulder-ex-al-interface__2__1"/>
       <child link="${prefix}_RMD-X8-Pro_MIR8_MIR1__1__1"/>
-      <axis xyz="-1.0 0.0 0.0"/>
+      <axis xyz="${sign * 1.0} 0.0 0.0"/>
       <limit upper="${PI}" lower="${-PI}" velocity="10.0" effort="100.0"/>
     </joint>
@@ -1479,5 +1479,5 @@
       <parent link="${prefix}_shoulder-ex-al-interface__1__1"/>
       <child link="${prefix}_RMD-X8-Pro_MIR8_MIR1__3__1"/>
-      <axis xyz="0.0 -1.0 0.0"/>
+      <axis xyz="0.0 ${sign*1.0} 0.0"/>
       <limit upper="${PI}" lower="${-PI}" velocity="10.0" effort="100.0"/>
     </joint>
@@ -1521,5 +1521,5 @@
       <parent link="${prefix}_RMD-X8-Pro_MIR8_MIR1__2__1"/>
       <child link="${prefix}_bicep-motor-mate_1"/>
-      <axis xyz="0.0 0.0 1.0"/>
+      <axis xyz="0.0 0.0 ${sign * 1.0}"/>
       <limit upper="${PI}" lower="${-PI}" velocity="10.0" effort="100.0"/>
       <dynamics damping="2.0"/>
@@ -1575,8 +1575,8 @@
           <velocity>10.0</velocity>
         </limit>
-        <!-- <dynamics>
+        <dynamics>
           <damping>10.0</damping>
           <friction>0.50</friction>
-        </dynamics> -->
+        </dynamics>
       </joint>
     </gazebo>
@@ -1650,8 +1650,8 @@
           <velocity>0.0</velocity> -->
         </limit>
-        <!-- <dynamics>
+        <dynamics>
           <damping>1.0</damping>
           <friction>0.5</friction>
-        </dynamics> -->
+        </dynamics>
       </joint>
       <joint name="${prefix}_Recolute48_gz" type="revolute">
@@ -1668,8 +1668,8 @@
           <velocity>0.0</velocity> -->
         </limit>
-        <!-- <dynamics>
+        <dynamics>
           <damping>2.0</damping>
           <friction>0.10</friction>
-        </dynamics> -->
+        </dynamics>
       </joint>
     </gazebo>
@@ -1729,5 +1729,5 @@
       <parent link="${prefix}_RMD-X8-Pro_MIR8_MIR1__4__1"/>
       <child link="${prefix}_shoulder-ex-al-interface_1"/>
-      <axis xyz="-0.000375 -1.0 0.0"/>
+      <axis xyz="0.0 ${sign * 1.0} 0.0"/>
       <limit upper="${PI}" lower="${-PI}" velocity="10.0" effort="100.0"/>
     </joint>
