Commit message: fix torso.xacro joint axis directions for correct rotation

File: dropbear-humanoid-robot/dropbear/urdf/gazebo/torso.xacro (robot description, xacro)
@@ -1716,5 +1716,5 @@
             <parent link="${prefix}_RMD-X10__1_Stator_1"/>
             <child link="${prefix}_RMD-X10__1_Rotor_1"/>
-            <axis xyz="0.0 0.0 -1.0"/>
+            <axis xyz="0.0 0.0 1.0"/>
             <limit upper="${PI}" lower="${-PI}" velocity="10.0" effort="10.0"/>
         </joint>
@@ -1733,5 +1733,5 @@
             <parent link="${prefix}_RMD-X10Stator_1"/>
             <child link="${prefix}_RMD-X10Rotot_1"/>
-            <axis xyz="0.0 0.0 1.0"/>
+            <axis xyz="0.0 0.0 -1.0"/>
             <limit upper="${PI}" lower="${-PI}" velocity="10.0" effort="10.0"/>
         </joint>
