Commit message: uncomment various macros and battery inclusion in dropbear_gz.urdf.xacro

File: dropbear-humanoid-robot/dropbear/urdf/gazebo/dropbear_gz.urdf.xacro (robot description, xacro)
@@ -17,5 +17,5 @@
     <!-- <xacro:include filename="$(find dropbear)/urdf/gazebo/head.xacro"/> -->
     <!-- Battery xacro -->
-    <!-- <xacro:include filename="$(find dropbear)/urdf/gazebo/battery.xacro"/> -->
+    <xacro:include filename="$(find dropbear)/urdf/gazebo/battery.xacro"/>
     <!-- ros2 control -->
     <xacro:include filename="$(find dropbear)/urdf/ros2_control/dropbear.ros2_control.xacro"/>
@@ -23,14 +23,14 @@
     <link name="world"/>
     <!-- Torso macro -->
-     <!-- <xacro:torso_macro prefix="torso">
-     </xacro:torso_macro> -->
+     <xacro:torso_macro prefix="torso">
+     </xacro:torso_macro>
     <!-- base_link to world joint -->
     <joint name="base_link_sim_world_joint" type="fixed">
-        <!-- <origin xyz="0.0 0.0 1.4" rpy="${PI/2} 0.0 0.0"/> -->
-        <origin xyz="0.0 0.0 1.4" rpy="${0} 0.0 0.0"/>
+        <origin xyz="0.0 0.0 1.4" rpy="${PI/2} 0.0 0.0"/>
+        <!-- <origin xyz="0.0 0.0 1.4" rpy="${0} 0.0 0.0"/> -->
         <parent link="world"/>
         <!-- Torso Base link -->
-        <!-- <child link="torso_base_link"/> -->
-        <child link="RL_base_link"/>
+        <child link="torso_base_link"/>
+        <!-- <child link="RL_base_link"/> -->
         <!-- <child link="RH_base_link"/> -->
     </joint>
@@ -45,38 +45,38 @@
     </xacro:head_macro> -->
     <!-- waist -->
-    <!-- <xacro:pelvicgirdle_macro prefix="PG" parent = "torso_lumbar-strap_1">
+    <xacro:pelvicgirdle_macro prefix="PG" parent = "torso_lumbar-strap_1">
         <origin xyz="-0.023253 -0.021955 0.0" rpy="${-PI/2} 0 0"/>
-    </xacro:pelvicgirdle_macro> -->
+    </xacro:pelvicgirdle_macro>
     <!-- Right Arm-->
-    <!-- <xacro:arm_macro prefix="RH" folder = "rightarm" parent = "torso_RMD-X10Rotot_1" sign = "1">
+    <xacro:arm_macro prefix="RH" folder = "rightarm" parent = "torso_RMD-X10Rotot_1" sign = "1">
         <origin xyz="0.0 0.0 0.0" rpy="0 0 0"/>
-    </xacro:arm_macro> -->
+    </xacro:arm_macro>
     <!-- <xacro:arm_macro prefix="RH" folder = "rightarm" parent = "RH_base_link" sign = "1">
         <origin xyz="0.0 0.0 0.0" rpy="0 0 0"/>
     </xacro:arm_macro> -->
     <!-- Left Arm -->
-    <!-- <xacro:arm_macro prefix="LH" folder = "leftarm" parent = "torso_RMD-X10__1_Rotor_1" sign = "-1">
+    <xacro:arm_macro prefix="LH" folder = "leftarm" parent = "torso_RMD-X10__1_Rotor_1" sign = "-1">
         <origin xyz="0.0 0.0 0.0" rpy="0 0 0"/>
-    </xacro:arm_macro> -->
+    </xacro:arm_macro>
     <!-- <xacro:arm_macro prefix="LH" folder = "leftarm" parent = "LH_base_link" sign = "-1">
         <origin xyz="0.0 0.0 0.0" rpy="0 0 0"/>
     </xacro:arm_macro> -->
     <!-- Right Leg -->
-    <!-- <xacro:leg_macro prefix = "RL" folder = "rightleg" parent = "PG_motor-yaw-cap_1" sign = "1">
+    <xacro:leg_macro prefix = "RL" folder = "rightleg" parent = "PG_motor-yaw-cap_1" sign = "1">
+        <origin xyz="0 0 0" rpy="${5/9 * PI} 0 0"/>
+    </xacro:leg_macro>
+    <!-- <xacro:leg_macro prefix = "RL" folder = "rightleg" parent = "RL_base_link" sign = "1">
         <origin xyz="0 0 0" rpy="${5/9 * PI} 0 0"/>
     </xacro:leg_macro> -->
-    <xacro:leg_macro prefix = "RL" folder = "rightleg" parent = "RL_base_link" sign = "1">
-        <origin xyz="0 0 0" rpy="${5/9 * PI} 0 0"/>
+    <!-- Left Leg -->
+    <xacro:leg_macro prefix = "LL" folder = "leftleg" parent = "PG_motor-yaw-cap__1__1" sign = "-1">
+        <origin xyz="0 0 0" rpy="${4/9 * PI} 0 0"/>
     </xacro:leg_macro>
-    <!-- Left Leg -->
-    <!-- <xacro:leg_macro prefix = "LL" folder = "leftleg" parent = "PG_motor-yaw-cap__1__1" sign = "-1">
-        <origin xyz="0 0 0" rpy="${4/9 * PI} 0 0"/>
-    </xacro:leg_macro> -->
     <!-- <xacro:leg_macro prefix = "LL" folder = "leftleg" parent = "RL_base_link" sign = "-1">
         <origin xyz="0.0 0.2 0.0" rpy="${4/9 * PI} 0 0"/>
     </xacro:leg_macro> -->
     <!-- Battery -->
-     <!-- <xacro:battery_macro parent = "torso_left-battery-mount_1">
+     <xacro:battery_macro parent = "torso_left-battery-mount_1">
         <origin xyz="0.08 -0.028115 0.03632" rpy="0 0 0"/>
-     </xacro:battery_macro> -->
+     </xacro:battery_macro>
 </robot>

Commit message: update base_link_sim_world_joint origin height to improve simulation accuracy

File: dropbear-humanoid-robot/dropbear/urdf/gazebo/dropbear_gz.urdf.xacro (robot description, xacro)
@@ -27,5 +27,5 @@
     <!-- base_link to world joint -->
     <joint name="base_link_sim_world_joint" type="fixed">
-        <origin xyz="0.0 0.0 1.4" rpy="${PI/2} 0.0 0.0"/>
+        <origin xyz="0.0 0.0 1.5" rpy="${PI/2} 0.0 0.0"/>
         <!-- <origin xyz="0.0 0.0 1.4" rpy="${0} 0.0 0.0"/> -->
         <parent link="world"/>

Commit message: add: include head xacro in URDF and add head macro definition

File: dropbear-humanoid-robot/dropbear/urdf/gazebo/dropbear_gz.urdf.xacro (robot description, xacro)
@@ -15,5 +15,5 @@
     <xacro:include filename="$(find dropbear)/urdf/gazebo/leg.xacro"/>
     <!-- Head xacro -->
-    <!-- <xacro:include filename="$(find dropbear)/urdf/gazebo/head.xacro"/> -->
+    <xacro:include filename="$(find dropbear)/urdf/gazebo/head.xacro"/>
     <!-- Battery xacro -->
     <xacro:include filename="$(find dropbear)/urdf/gazebo/battery.xacro"/>
@@ -41,7 +41,7 @@
     </joint> -->
     <!-- Head -->
-    <!-- <xacro:head_macro prefix="head" parent = "torso_base_link">
+    <xacro:head_macro prefix="head" parent = "torso_base_link">
         <origin xyz="0.0985 0.0798 0.069747" rpy="0 ${PI/2} 0"/>
-    </xacro:head_macro> -->
+    </xacro:head_macro>
     <!-- waist -->
     <xacro:pelvicgirdle_macro prefix="PG" parent = "torso_lumbar-strap_1">
