Commit message: add: include head xacro in URDF and add head macro definition

File: dropbear-humanoid-robot/dropbear/urdf/gazebo/head.xacro (robot description, xacro)
@@ -6,6 +6,6 @@
       <inertial>
         <origin xyz="-2.930562105762924e-07 0.022659839097962126 -0.03078226707220777" rpy="0 0 0"/>
-        <mass value="0.03431683927055112"/>
-        <inertia ixx="2e-05" iyy="2.5e-05" izz="9e-06" ixy="-0.0" iyz="2e-06" ixz="-0.0"/>
+        <mass value="0.0343168392705511"/>
+        <inertia ixx="2.02171782450449e-05" iyy="2.48368303351022e-05" izz="8.97645024047333e-06" ixy="-8.139786587813003e-13" iyz="2.29034767095513e-06" ixz="-2.046957330199828e-12"/>
       </inertial>
       <visual>
@@ -26,6 +26,6 @@
       <inertial>
         <origin xyz="-2.660500832418755e-07 0.006823295397768353 -0.010000400049690328" rpy="0 0 0"/>
-        <mass value="0.03822624114902457"/>
-        <inertia ixx="5e-06" iyy="2.7e-05" izz="2.3e-05" ixy="-0.0" iyz="-0.0" ixz="0.0"/>
+        <mass value="0.0382262411490246"/>
+        <inertia ixx="5.21422282842468e-06" iyy="2.68511514044845e-05" izz="2.2970122979932e-05" ixy="-8.124167788156611e-12" iyz="-5.313974737672367e-12" ixz="1.868346493141826e-11"/>
       </inertial>
       <visual>
@@ -46,6 +46,6 @@
       <inertial>
         <origin xyz="-0.015500289972000925 -0.01905943358743986 -0.015500434949509062" rpy="0 0 0"/>
-        <mass value="0.06723933852178482"/>
-        <inertia ixx="1.8e-05" iyy="1.9e-05" izz="1.8e-05" ixy="-0.0" iyz="0.0" ixz="-0.0"/>
+        <mass value="0.0672393385217848"/>
+        <inertia ixx="1.84430010390104e-05" iyy="1.85822752361295e-05" izz="1.84430010331934e-05" ixy="-4.293440603042598e-17" iyz="2.168404344971009e-19" ixz="-4.336808689942018e-19"/>
       </inertial>
       <visual>
@@ -66,6 +66,6 @@
       <inertial>
         <origin xyz="-0.015500289972022074 -0.01905943358743986 -0.015500434949530267" rpy="0 0 0"/>
-        <mass value="0.06723933852178482"/>
-        <inertia ixx="1.8e-05" iyy="1.9e-05" izz="1.8e-05" ixy="0.0" iyz="0.0" ixz="0.0"/>
+        <mass value="0.0672393385217848"/>
+        <inertia ixx="1.8443001033193e-05" iyy="1.85822752361287e-05" izz="1.84430010390126e-05" ixy="0" iyz="4.250072516143177e-17" ixz="0"/>
       </inertial>
       <visual>
@@ -86,6 +86,6 @@
       <inertial>
         <origin xyz="-0.020320289972009742 -0.00017258686465915218 -0.035196434949503426" rpy="0 0 0"/>
-        <mass value="0.08770478761203049"/>
-        <inertia ixx="6.6e-05" iyy="0.000126" izz="6.6e-05" ixy="0.0" iyz="0.0" ixz="0.0"/>
+        <mass value="0.0877047876120305"/>
+        <inertia ixx="6.61769319433791e-05" iyy="0.000126427648128685" izz="6.61769319420177e-05" ixy="1.734723475976807e-18" iyz="3.794707603699266e-19" ixz="1.179069862577986e-15"/>
       </inertial>
       <visual>
@@ -106,6 +106,6 @@
       <inertial>
         <origin xyz="-0.03463441624017194 0.00209942994352158 -0.020706224659481694" rpy="0 0 0"/>
-        <mass value="0.06395878873611698"/>
-        <inertia ixx="0.0001" iyy="0.000191" izz="0.000101" ixy="-0.0" iyz="0.0" ixz="-0.0"/>
+        <mass value="0.063958788736117"/>
+        <inertia ixx="0.000100418070794671" iyy="0.000191106026686862" izz="0.000101099832749464" ixy="-2.1488139835199e-09" iyz="1.85453404233848e-07" ixz="-5.83855603187439e-09"/>
       </inertial>
       <visual>
@@ -126,6 +126,6 @@
       <inertial>
         <origin xyz="0.01713833984577129 -0.0023401609020378134 -0.03335951621717591" rpy="0 0 0"/>
-        <mass value="0.03431683927055112"/>
-        <inertia ixx="1.2e-05" iyy="2.5e-05" izz="1.7e-05" ixy="2e-06" iyz="-1e-06" ixz="5e-06"/>
+        <mass value="0.0343168392705511"/>
+        <inertia ixx="1.17866340143334e-05" iyy="2.48368303351031e-05" izz="1.74069944711835e-05" ixy="1.98349967353486e-06" iyz="-1.14517313055135e-06" ixz="4.86737902797394e-06"/>
       </inertial>
       <visual>
@@ -146,6 +146,6 @@
       <inertial>
         <origin xyz="-0.03745891670562651 -0.0023401609020367586 0.0018374784408524414" rpy="0 0 0"/>
-        <mass value="0.03431683927055112"/>
-        <inertia ixx="1.2e-05" iyy="2.5e-05" izz="1.7e-05" ixy="-2e-06" iyz="-1e-06" ixz="-5e-06"/>
+        <mass value="0.0343168392705511"/>
+        <inertia ixx="1.17866304688991e-05" iyy="2.48368303351024e-05" izz="1.74069980166196e-05" ixy="-1.98349885955598e-06" iyz="-1.14517454040368e-06" ixz="-4.86737698101647e-06"/>
       </inertial>
       <visual>
@@ -166,6 +166,6 @@
       <inertial>
         <origin xyz="-0.05369329673498335 0.029021748898090435 -0.031000429563639173" rpy="0 0 0"/>
-        <mass value="0.09089909699962714"/>
-        <inertia ixx="0.000139" iyy="0.000258" izz="0.000139" ixy="-0.0" iyz="-0.0" ixz="-0.0"/>
+        <mass value="0.0908990969996271"/>
+        <inertia ixx="0.000139021398765956" iyy="0.000257606464021122" izz="0.000139021638500429" ixy="-5.573025981669977e-12" iyz="-3.025921527233244e-13" ixz="-1.33157682254657e-10"/>
       </inertial>
       <visual>
@@ -186,6 +186,6 @@
       <inertial>
         <origin xyz="-0.017752035586700965 -0.02347097657744404 0.005425623888361868" rpy="0 0 0"/>
-        <mass value="0.014270297097400294"/>
-        <inertia ixx="2e-06" iyy="1e-06" izz="3e-06" ixy="-1e-06" iyz="0.0" ixz="0.0"/>
+        <mass value="0.0142702970974003"/>
+        <inertia ixx="2.11854674702863e-06" iyy="1.31034225113913e-06" izz="2.79505580106851e-06" ixy="-5.56425019936969e-07" iyz="1.15254347270033e-07" ixz="4.19538481116912e-07"/>
       </inertial>
       <visual>
@@ -206,6 +206,6 @@
       <inertial>
         <origin xyz="-0.013806611207024755 -0.022230262084818597 0.012754435460634692" rpy="0 0 0"/>
-        <mass value="0.016008852298185192"/>
-        <inertia ixx="2e-06" iyy="1e-06" izz="3e-06" ixy="1e-06" iyz="-0.0" ixz="0.0"/>
+        <mass value="0.0160088522981852"/>
+        <inertia ixx="2.34534575173438e-06" iyy="1.40164111174057e-06" izz="3.06606262275542e-06" ixy="6.18530934732024e-07" iyz="-1.44549164161862e-07" ixz="4.53978402064964e-07"/>
       </inertial>
       <visual>
@@ -226,6 +226,6 @@
       <inertial>
         <origin xyz="-0.0041424710537947 -0.022230262084817515 -0.018333211458883378" rpy="0 0 0"/>
-        <mass value="0.016008852298185286"/>
-        <inertia ixx="3e-06" iyy="1e-06" izz="2e-06" ixy="-0.0" iyz="1e-06" ixz="0.0"/>
+        <mass value="0.0160088522981853"/>
+        <inertia ixx="3.27904023395687e-06" iyy="1.40164111182438e-06" izz="2.13236814061474e-06" ixy="-1.8408221772793e-07" iyz="6.07938084585139e-07" ixz="8.5090356813296e-08"/>
       </inertial>
       <visual>
@@ -246,6 +246,6 @@
       <inertial>
         <origin xyz="0.004141891109750773 -0.022230262084818653 -0.01766614498065596" rpy="0 0 0"/>
-        <mass value="0.016008852298185283"/>
-        <inertia ixx="3e-06" iyy="1e-06" izz="2e-06" ixy="0.0" iyz="-1e-06" ixz="0.0"/>
+        <mass value="0.0160088522981853"/>
+        <inertia ixx="3.2790402339573e-06" iyy="1.40164111182579e-06" izz="2.13236814061756e-06" ixy="1.8408221772793e-07" iyz="-6.07938084585275e-07" ixz="8.50903568132689e-08"/>
       </inertial>
       <visual>
@@ -266,6 +266,6 @@
       <inertial>
         <origin xyz="0.01322833473847393 -0.02223026208481757 0.012420902235982481" rpy="0 0 0"/>
-        <mass value="0.01600885229818528"/>
-        <inertia ixx="2e-06" iyy="1e-06" izz="3e-06" ixy="0.0" iyz="0.0" ixz="-1e-06"/>
+        <mass value="0.0160088522981853"/>
+        <inertia ixx="2.49272657456873e-06" iyy="1.40164111182427e-06" izz="2.91868180000445e-06" ixy="4.34448716314867e-07" iyz="4.63388919229692e-07" ixz="-5.39068759728735e-07"/>
       </inertial>
       <visual>
@@ -286,6 +286,6 @@
       <inertial>
         <origin xyz="0.0179482123364042 -0.022230262084817543 0.00557947113525567" rpy="0 0 0"/>
-        <mass value="0.016008852298185283"/>
-        <inertia ixx="2e-06" iyy="1e-06" izz="3e-06" ixy="-0.0" iyz="-0.0" ixz="-1e-06"/>
+        <mass value="0.0160088522981853"/>
+        <inertia ixx="2.49272657456802e-06" iyy="1.40164111182427e-06" izz="2.91868180000293e-06" ixy="-4.34448716315843e-07" iyz="-4.63388919229597e-07" ixz="-5.39068759728898e-07"/>
       </inertial>
       <visual>
@@ -306,6 +306,6 @@
       <inertial>
         <origin xyz="-0.01187821563234115 0.0004424088449214436 0.020772195154224186" rpy="0 0 0"/>
-        <mass value="0.032098307887792374"/>
-        <inertia ixx="6e-06" iyy="8e-06" izz="2e-06" ixy="0.0" iyz="-0.0" ixz="-0.0"/>
+        <mass value="0.0320983078877924"/>
+        <inertia ixx="6.18689971729615e-06" iyy="8.16520250959728e-06" izz="2.17902054183792e-06" ixy="3.0321370657338e-09" iyz="-1.01914171671364e-07" ixz="-1.54181321521856e-08"/>
       </inertial>
       <visual>
@@ -326,6 +326,6 @@
       <inertial>
         <origin xyz="0.008660211834631892 0.006823295397769463 0.004999561783391355" rpy="0 0 0"/>
-        <mass value="0.03822624114902457"/>
-        <inertia ixx="1.9e-05" iyy="2.7e-05" izz="1e-05" ixy="-0.0" iyz="0.0" ixz="8e-06"/>
+        <mass value="0.0382262411490246"/>
+        <inertia ixx="1.85311641224101e-05" iyy="2.68511514044843e-05" izz="9.65318168594546e-06" ixy="-8.664120853055235e-12" iyz="4.378748069428645e-12" ixz="7.68852095740021e-06"/>
       </inertial>
       <visual>
@@ -346,6 +346,6 @@
       <inertial>
         <origin xyz="-0.008660731330417892 0.006823295397769463 0.004999526883572445" rpy="0 0 0"/>
-        <mass value="0.03822624114902457"/>
-        <inertia ixx="1.9e-05" iyy="2.7e-05" izz="1e-05" ixy="-0.0" iyz="0.0" ixz="-8e-06"/>
+        <mass value="0.0382262411490246"/>
+        <inertia ixx="1.85311317616992e-05" iyy="2.68511514044832e-05" izz="9.65321404665636e-06" ixy="-5.399530648986239e-13" iyz="9.692722658023213e-12" ixz="-7.68853964086547e-06"/>
       </inertial>
       <visual>
@@ -366,6 +366,6 @@
       <inertial>
         <origin xyz="0.021173169649522317 -0.019059433587438862 -0.0056737998548819085" rpy="0 0 0"/>
-        <mass value="0.06723933852178482"/>
-        <inertia ixx="1.8e-05" iyy="1.9e-05" izz="1.8e-05" ixy="0.0" iyz="-0.0" ixz="-0.0"/>
+        <mass value="0.0672393385217848"/>
+        <inertia ixx="1.84430010346467e-05" iyy="1.85822752361282e-05" izz="1.84430010375554e-05" ixy="2.125036258071589e-17" iyz="-3.686456793040166e-17" ixz="-2.519177629087960e-15"/>
       </inertial>
       <visual>
@@ -386,6 +386,6 @@
       <inertial>
         <origin xyz="0.0056731696496243045 -0.019059433587472863 0.021172929955841774" rpy="0 0 0"/>
-        <mass value="0.06723933852178482"/>
-        <inertia ixx="1.8e-05" iyy="1.9e-05" izz="1.8e-05" ixy="-0.0" iyz="-0.0" ixz="0.0"/>
+        <mass value="0.0672393385217848"/>
+        <inertia ixx="1.8443001037555e-05" iyy="1.85822752361274e-05" izz="1.8443001034648e-05" ixy="-3.729655473350135e-17" iyz="-2.119615247209161e-17" ixz="2.519143747770070e-15"/>
       </inertial>
       <visual>
@@ -406,6 +406,6 @@
       <inertial>
         <origin xyz="-0.005673749593571531 -0.01905943358744086 0.02117292995588415" rpy="0 0 0"/>
-        <mass value="0.06723933852178482"/>
-        <inertia ixx="1.8e-05" iyy="1.9e-05" izz="1.8e-05" ixy="-0.0" iyz="-0.0" ixz="0.0"/>
+        <mass value="0.0672393385217848"/>
+        <inertia ixx="1.84430010346467e-05" iyy="1.85822752361269e-05" izz="1.84430010375554e-05" ixy="-2.168404344971009e-17" iyz="-3.686287386450715e-17" ixz="2.519035327552821e-15"/>
       </inertial>
       <visual>
@@ -426,6 +426,6 @@
       <inertial>
         <origin xyz="-0.021173749593575764 -0.019059433587443803 -0.005673799854911454" rpy="0 0 0"/>
-        <mass value="0.06723933852178482"/>
-        <inertia ixx="1.8e-05" iyy="1.9e-05" izz="1.8e-05" ixy="-0.0" iyz="0.0" ixz="-0.0"/>
+        <mass value="0.0672393385217848"/>
+        <inertia ixx="1.84430010375554e-05" iyy="1.85822752361287e-05" izz="1.84430010346463e-05" ixy="-3.729655473350135e-17" iyz="2.128424389860606e-17" ixz="-2.519177629087960e-15"/>
       </inertial>
       <visual>
@@ -446,6 +446,6 @@
       <inertial>
         <origin xyz="-3.0642435633332354e-07 -0.001802890975442284 -4.0069029630385167e-07" rpy="0 0 0"/>
-        <mass value="0.0019034168312865901"/>
-        <inertia ixx="75.91e-09" iyy="71.51e-09" izz="82.56e-09" ixy="0.0" iyz="0.0" ixz="-7.0e-09"/>
+        <mass value="0.00190341683128659"/>
+        <inertia ixx="7.59046150555949e-08" iyy="7.15058292314534e-08" izz="8.25591352973242e-08" ixy="1.043864430658181e-13" iyz="-2.146755131516090e-13" ixz="-7.00721363018056e-09"/>
       </inertial>
       <visual>
@@ -466,6 +466,6 @@
       <inertial>
         <origin xyz="-0.004226364224141521 -3.831484196581414e-08 -0.002671317839583298" rpy="0 0 0"/>
-        <mass value="0.0009727380393185158"/>
-        <inertia ixx="14.27e-09" iyy="19.21e-09" izz="16.13e-09" ixy="2.27e-10" iyz="-1.34e-09" ixz="-3.25e-10"/>
+        <mass value="0.000972738039318516"/>
+        <inertia ixx="1.48510965590436e-08" iyy="1.89536797372714e-08" izz="1.58104434504197e-08" ixy="8.5682910457496e-10" iyz="-1.35536961805103e-09" ixz="-1.01018993036329e-09"/>
       </inertial>
       <visual>
@@ -486,6 +486,6 @@
       <inertial>
         <origin xyz="-0.0016515827964225793 0.012920991301931556 0.0020304100943668163" rpy="0 0 0"/>
-        <mass value="0.0016579387604439215"/>
-        <inertia ixx="8.233e-08" iyy="6.909e-08" izz="6.775e-08" ixy="2.663e-08" iyz="-7.07e-10" ixz="-1.151e-08"/>
+        <mass value="0.00165793876044392"/>
+        <inertia ixx="7.87567114191468e-08" iyy="6.85285465555218e-08" izz="7.1887778374367e-08" ixy="6.01452920535308e-10" iyz="-2.44551611159629e-10" ixz="6.80340347335954e-09"/>
       </inertial>
       <visual>
@@ -506,6 +506,6 @@
       <inertial>
         <origin xyz="0.008780592596962566 0.03773249316571298 -0.01622185986170563" rpy="0 0 0"/>
-        <mass value="0.04021238596594936"/>
-        <inertia ixx="3.2e-05" iyy="7e-06" izz="2.9e-05" ixy="-6e-06" iyz="1.2e-05" ixz="3e-06"/>
+        <mass value="0.0402123859659494"/>
+        <inertia ixx="3.22135153795742e-05" iyy="6.75415269858412e-06" izz="2.86963733738812e-05" ixy="-6.2638445207996e-06" iyz="1.1571807315945e-05" ixz="2.69286889615847e-06"/>
       </inertial>
       <visual>
@@ -526,6 +526,6 @@
       <inertial>
         <origin xyz="0.003050602859310525 0.013107335161964245 -0.0056355991364953895" rpy="0 0 0"/>
-        <mass value="0.02595839104798968"/>
-        <inertia ixx="1e-06" iyy="1e-06" izz="1e-06" ixy="0.0" iyz="-0.0" ixz="-0.0"/>
+        <mass value="0.0259583910479897"/>
+        <inertia ixx="1.04482267874984e-06" iyy="1.40990448271048e-06" izz="1.09525773804922e-06" ixy="8.98221896935983e-08" iyz="-1.65937239508926e-07" ixz="-3.86151594376598e-08"/>
       </inertial>
       <visual>
@@ -547,5 +547,5 @@
         <origin xyz="0.009492189078626478 0.040788178126711705 -0.017535202787712437" rpy="0 0 0"/>
         <mass value="0.0152025703381625"/>
-        <inertia ixx="1.7e-05" iyy="4e-06" izz="1.5e-05" ixy="-3e-06" iyz="6e-06" ixz="1e-06"/>
+        <inertia ixx="1.70263578660154e-05" iyy="4.01496000576487e-06" izz="1.52288684850605e-05" ixy="-3.20123383127209e-06" iyz="5.91394964386213e-06" ixz="1.37623196363882e-06"/>
       </inertial>
       <visual>
@@ -566,6 +566,6 @@
       <inertial>
         <origin xyz="0.001363586099866032 0.0058591437992934915 -0.002518532432421408" rpy="0 0 0"/>
-        <mass value="0.0016579387604439215"/>
-        <inertia ixx="8.233e-08" iyy="6.909e-08" izz="6.775e-08" ixy="2.663e-08" iyz="-7.07e-10" ixz="-1.151e-08"/>
+        <mass value="0.00165793876044392"/>
+        <inertia ixx="6.85476867241706e-08" iyy="7.02048764479374e-08" izz="8.04204731770411e-08" ixy="1.57657827044181e-09" iyz="4.18236807697612e-09" ixz="3.54482186936826e-09"/>
       </inertial>
       <visual>
@@ -586,6 +586,6 @@
       <inertial>
         <origin xyz="-0.0004911913800194068 -0.0021099981730251316 0.0009073107632914246" rpy="0 0 0"/>
-        <mass value="0.00016378169700714462"/>
-        <inertia ixx="1.244e-09" iyy="1.568e-09" izz="1.142e-09" ixy="-2.08e-10" iyz="5e-12" ixz="-3.0e-12"/>
+        <mass value="0.000163781697007145"/>
+        <inertia ixx="1.16509020847162e-09" iyy="1.56805759278815e-09" izz="1.22075907914391e-09" ixy="9.914329433629512e-11" iyz="-1.83157009534047e-10" ixz="-4.262236269847675e-11"/>
       </inertial>
       <visual>
@@ -606,6 +606,6 @@
       <inertial>
         <origin xyz="-0.004714550703255438 0.0014502030420020882 0.0008203215430236804" rpy="0 0 0"/>
-        <mass value="0.0009727380393185158"/>
-        <inertia ixx="14.27e-09" iyy="19.21e-09" izz="16.13e-09" ixy="2.27e-10" iyz="-1.34e-09" ixz="-3.25e-10"/>
+        <mass value="0.000972738039318516"/>
+        <inertia ixx="1.5956686999643e-08" iyy="1.9393580168254e-08" izz="1.42649525788148e-08" ixy="1.11343738653016e-09" iyz="-1.90124883084341e-10" ixz="-3.02519022134825e-10"/>
       </inertial>
       <visual>
@@ -626,6 +626,6 @@
       <inertial>
         <origin xyz="-0.0013771103535349938 0.010094796803556981 -0.00787380305235634" rpy="0 0 0"/>
-        <mass value="0.0014232382644525146"/>
-        <inertia ixx="65.84e-09" iyy="63.94e-09" izz="73.94e-09" ixy="-3.0e-12" iyz="-2.0e-12" ixz="6.53e-09"/>
+        <mass value="0.00142323826445251"/>
+        <inertia ixx="7.71186168343853e-08" iyy="6.39366996782876e-08" izz="6.26637183269083e-08" ixy="1.064945267556614e-11" iyz="-7.241465376321146e-13" ixz="-2.59152694047143e-09"/>
       </inertial>
       <visual>
@@ -646,6 +646,6 @@
       <inertial>
         <origin xyz="-2.8817588032525876e-07 -0.001802890975445226 -4.730412566378295e-07" rpy="0 0 0"/>
-        <mass value="0.0019034168312865901"/>
-        <inertia ixx="75.91e-09" iyy="71.51e-09" izz="82.56e-09" ixy="0.0" iyz="0.0" ixz="-7.0e-09"/>
+        <mass value="0.00190341683128659"/>
+        <inertia ixx="7.19067090216999e-08" iyy="7.15058292314534e-08" izz="8.65570413312192e-08" ixy="-1.347454591481279e-14" iyz="2.383286574819329e-13" ixz="-2.55218407959311e-09"/>
       </inertial>
       <visual>
@@ -666,6 +666,6 @@
       <inertial>
         <origin xyz="-0.004930302973391587 1.0162823481374428e-07 -0.0008343581172669257" rpy="0 0 0"/>
-        <mass value="0.0009727380393185158"/>
-        <inertia ixx="14.27e-09" iyy="19.21e-09" izz="16.13e-09" ixy="2.27e-10" iyz="-1.34e-09" ixz="-3.25e-10"/>
+        <mass value="0.000972738039318516"/>
+        <inertia ixx="1.42675062542425e-08" iyy="1.92135974511829e-08" izz="1.61341160413465e-08" ixy="2.27095967688707e-10" iyz="-1.34203495749462e-09" ixz="-3.2517451800879e-10"/>
       </inertial>
       <visual>
@@ -686,6 +686,6 @@
       <inertial>
         <origin xyz="-0.0009468839590772715 0.00655068127235281 -0.011401971728201676" rpy="0 0 0"/>
-        <mass value="0.0016579387604439215"/>
-        <inertia ixx="8.233e-08" iyy="6.909e-08" izz="6.775e-08" ixy="2.663e-08" iyz="-7.07e-10" ixz="-1.151e-08"/>
+        <mass value="0.00165793876044392"/>
+        <inertia ixx="8.19564327164812e-08" iyy="6.95081725009077e-08" izz="6.7708431131789e-08" ixy="3.5325259652459e-09" iyz="-2.05194968740157e-10" ixz="1.08014405327483e-09"/>
       </inertial>
       <visual>
@@ -706,6 +706,6 @@
       <inertial>
         <origin xyz="-0.008788805871513428 0.03774724464684516 -0.016182757997603645" rpy="0 0 0"/>
-        <mass value="0.04021238596594936"/>
-        <inertia ixx="3.2e-05" iyy="7e-06" izz="2.9e-05" ixy="6e-06" iyz="1.2e-05" ixz="-3e-06"/>
+        <mass value="0.0402123859659494"/>
+        <inertia ixx="3.22110011645789e-05" iyy="6.73307272578165e-06" izz="2.87199675616783e-05" ixy="6.27169862927929e-06" iyz="1.15488532160547e-05" ixz="-2.68879137858141e-06"/>
       </inertial>
       <visual>
@@ -726,6 +726,6 @@
       <inertial>
         <origin xyz="-0.003052434418171046 0.013112632288605985 -0.005621967312849169" rpy="0 0 0"/>
-        <mass value="0.02595839104798968"/>
-        <inertia ixx="1e-06" iyy="1e-06" izz="1e-06" ixy="-0.0" iyz="-0.0" ixz="0.0"/>
+        <mass value="0.0259583910479897"/>
+        <inertia ixx="1.04485873392106e-06" iyy="1.41020676558759e-06" izz="1.09491940000176e-06" ixy="-8.99348134832329e-08" iyz="-1.65608082614314e-07" ixz="3.85566933235482e-08"/>
       </inertial>
       <visual>
@@ -747,5 +747,5 @@
         <origin xyz="-0.00950027695477021 0.04080458802102564 -0.017493562988578126" rpy="0 0 0"/>
         <mass value="0.0152025703381625"/>
-        <inertia ixx="1.7e-05" iyy="4e-06" izz="1.5e-05" ixy="3e-06" iyz="6e-06" ixz="-1e-06"/>
+        <inertia ixx="1.70250729301238e-05" iyy="4.0041867637999e-06" izz="1.52409266629168e-05" ixy="3.20524779363137e-06" iyz="5.90221860249884e-06" ixz="-1.37414808247689e-06"/>
       </inertial>
       <visual>
@@ -766,6 +766,6 @@
       <inertial>
         <origin xyz="-0.0013645713509783663 0.00586082319007015 -0.0025132403706452783" rpy="0 0 0"/>
-        <mass value="0.0016579387604439215"/>
-        <inertia ixx="8.233e-08" iyy="6.909e-08" izz="6.775e-08" ixy="2.663e-08" iyz="-7.07e-10" ixz="-1.151e-08"/>
+        <mass value="0.00165793876044392"/>
+        <inertia ixx="8.23328616325021e-08" iyy="6.90904458543673e-08" izz="6.77497288622018e-08" ixy="2.66292977856842e-09" iyz="-7.0705185933362e-10" ixz="-1.15148979684771e-09"/>
       </inertial>
       <visual>
@@ -786,6 +786,6 @@
       <inertial>
         <origin xyz="0.0004913438048894381 -0.002110638420285813 0.000904783677481466" rpy="0 0 0"/>
-        <mass value="0.00016378169700714462"/>
-        <inertia ixx="1.244e-09" iyy="1.568e-09" izz="1.142e-09" ixy="-2.08e-10" iyz="5e-12" ixz="-3.0e-12"/>
+        <mass value="0.000163781697007145"/>
+        <inertia ixx="1.16513002424994e-09" iyy="1.56839124206287e-09" izz="1.22038561408938e-09" ixy="-9.926760161411958e-11" iyz="-1.82793702609653e-10" ixz="4.255782796210982e-11"/>
       </inertial>
       <visual>
@@ -806,6 +806,6 @@
       <inertial>
         <origin xyz="-3.210636296130387e-06 -0.0019705200384394286 -0.004594639231787129" rpy="0 0 0"/>
-        <mass value="0.0009727380393185158"/>
-        <inertia ixx="14.27e-09" iyy="19.21e-09" izz="16.13e-09" ixy="2.27e-10" iyz="-1.34e-09" ixz="-3.25e-10"/>
+        <mass value="0.000972738039318516"/>
+        <inertia ixx="1.4212482294692e-08" iyy="1.91035122500962e-08" izz="1.62992252019498e-08" ixy="2.269160497998519e-12" iyz="-1.47426492837938e-09" ixz="-4.677826526198851e-14"/>
       </inertial>
       <visual>
@@ -826,6 +826,6 @@
       <inertial>
         <origin xyz="-0.007994368928315204 0.010094151077657335 9.279386893601416e-07" rpy="0 0 0"/>
-        <mass value="0.0014232382644525146"/>
-        <inertia ixx="65.84e-09" iyy="63.94e-09" izz="73.94e-09" ixy="-3.0e-12" iyz="-2.0e-12" ixz="6.53e-09"/>
+        <mass value="0.00142323826445251"/>
+        <inertia ixx="6.22131468412977e-08" iyy="6.39366921736977e-08" izz="7.75691958245672e-08" ixy="9.764173383676120e-13" iyz="2.856308677636431e-12" ixz="5.885762099325665e-12"/>
       </inertial>
       <visual>
@@ -846,6 +846,6 @@
       <inertial>
         <origin xyz="2.425383274773374e-07 -0.0018028909754462807 1.6296356755100133e-07" rpy="0 0 0"/>
-        <mass value="0.0019034168312865901"/>
-        <inertia ixx="75.91e-09" iyy="71.51e-09" izz="82.56e-09" ixy="0.0" iyz="0.0" ixz="-7.0e-09"/>
+        <mass value="0.00190341683128659"/>
+        <inertia ixx="7.16072026664091e-08" iyy="7.15058292314534e-08" izz="8.68565476865642e-08" ixy="4.827892642958465e-14" iyz="2.337760840363973e-13" ixz="1.42690990802672e-09"/>
       </inertial>
       <visual>
@@ -866,6 +866,6 @@
       <inertial>
         <origin xyz="-0.004978762007825321 -4.937069585098097e-08 0.0004620643261550869" rpy="0 0 0"/>
-        <mass value="0.0009727380393185158"/>
-        <inertia ixx="14.27e-09" iyy="19.21e-09" izz="16.13e-09" ixy="2.27e-10" iyz="-1.34e-09" ixz="-3.25e-10"/>
+        <mass value="0.000972738039318516"/>
+        <inertia ixx="1.4229514241373e-08" iyy="1.91939383707891e-08" izz="1.61917671345421e-08" ixy="1.27715555734993e-10" iyz="1.37673188732768e-09" ixz="1.83612823701973e-10"/>
       </inertial>
       <visual>
@@ -886,6 +886,6 @@
       <inertial>
         <origin xyz="-0.0017065991424044524 0.006495882954367288 0.011343866964438839" rpy="0 0 0"/>
-        <mass value="0.0016579387604439215"/>
-        <inertia ixx="8.233e-08" iyy="6.909e-08" izz="6.775e-08" ixy="2.663e-08" iyz="-7.07e-10" ixz="-1.151e-08"/>
+        <mass value="0.00165793876044392"/>
+        <inertia ixx="8.20983716009993e-08" iyy="6.94417553190134e-08" izz="6.76329094290466e-08" ixy="3.39822253347358e-09" iyz="4.70339885215196e-10" ixz="-2.185043489367157e-11"/>
       </inertial>
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